File: hardware/board/harp_lick_detector_capactive/sine_wave_source.kicad_sch (KiCad schematic)
At the start: 12 parts

Commit message: complete bom draft
Parts:
- added C? (x2): (no value), symbol Device:C
Connections:
- net +5V: now also C?.1
- net -5V: now also C?.2
- net GNDA: now also C?.1, C?.2
Other:
- note added: "ADA4807-2 Bypass Caps"
- moved on the sheet: U3C

Commit message: add usb isolator
Parts:
- C?: value (none) -> 10uF
- C? (x4): value (none) -> 100nF
- C? (x2): value (none) -> 10nF
- C?: value (none) -> 1nF
- R?: value (none) -> 68K
- R?: value (none) -> 150K
- R?: value (none) -> 5.1
- U3: value (none) -> ADA4807-2ARM
- U4: value (none) -> AD9833xRM
- X1: value (none) -> ASE-25.000MHZ-L-C-T; footprint (none) -> Crystal:Crystal_SMD_Abracon_ABM8G-4Pin_3.2x2.5mm
Changed lines of the file:
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@@
       (effects (font (size 1.27 1.27)) (justify left))
     )
-    (property "Value" "" (id 1) (at 44.45 176.53 0)
+    (property "Value" "10uF" (id 1) (at 44.45 176.53 0)
       (effects (font (size 1.27 1.27)) (justify left))
     )
@@
     (in_bom yes) (on_board yes)
     (property "Reference" "X1" (id 0) (at 99.06 91.44 0))
-    (property "Value" "" (id 1) (at 111.76 104.14 0))
-    (property "Footprint" "" (id 2) (at 120.65 106.68 0)
+    (property "Value" "ASE-25.000MHZ-L-C-T" (id 1) (at 111.76 104.14 0))
+    (property "Footprint" "Crystal:Crystal_SMD_Abracon_ABM8G-4Pin_3.2x2.5mm" (id 2) (at 120.65 106.68 0)
       (effects (font (size 1.27 1.27)) hide)
     )
@@
     (in_bom yes) (on_board yes)
     (property "Reference" "U4" (id 0) (at 124.46 81.28 0))
-    (property "Value" "" (id 1) (at 144.78 81.28 0))
+    (property "Value" "AD9833xRM" (id 1) (at 144.78 81.28 0))
     (property "Footprint" "" (id 2) (at 135.89 107.95 0)
       (effects (font (size 1.27 1.27)) hide)
@@
       (effects (font (size 1.27 1.27)) (justify left))
     )
-    (property "Value" "" (id 1) (at 133.35 72.39 90)
+    (property "Value" "100nF" (id 1) (at 133.35 72.39 90)
       (effects (font (size 1.27 1.27)) (justify left))
     )
@@
       (effects (font (size 1.27 1.27)) (justify left))
     )
-    (property "Value" "" (id 1) (at 30.48 176.53 0)
+    (property "Value" "10nF" (id 1) (at 30.48 176.53 0)
       (effects (font (size 1.27 1.27)) (justify left))
     )
@@
     (in_bom yes) (on_board yes) (fields_autoplaced)
     (property "Reference" "U3" (id 0) (at 191.77 100.33 0))
-    (property "Value" "" (id 1) (at 191.77 102.87 0))
+    (property "Value" "ADA4807-2ARM" (id 1) (at 191.77 102.87 0))
     (property "Footprint" "" (id 2) (at 191.77 110.49 0)
       (effects (font (size 1.27 1.27)) hide)
@@
       (effects (font (size 1.27 1.27)) (justify left))
     )
-    (property "Value" "" (id 1) (at 67.31 167.64 0)
+    (property "Value" "100nF" (id 1) (at 67.31 167.64 0)
       (effects (font (size 1.27 1.27)) (justify left))
     )
@@
       (effects (font (size 1.27 1.27)) (justify right))
     )
-    (property "Value" "" (id 1) (at 157.48 85.0899 0)
+    (property "Value" "10nF" (id 1) (at 157.48 85.0899 0)
       (effects (font (size 1.27 1.27)) (justify right))
     )
@@
       (effects (font (size 1.27 1.27)) (justify left))
     )
-    (property "Value" "" (id 1) (at 63.5 175.2599 0)
+    (property "Value" "ADA4807-2ARM" (id 1) (at 63.5 175.2599 0)
       (effects (font (size 1.27 1.27)) (justify left) hide)
     )
@@
       (effects (font (size 1.27 1.27)) (justify left))
     )
-    (property "Value" "" (id 1) (at 172.72 104.14 90)
+    (property "Value" "68K" (id 1) (at 172.72 104.14 90)
       (effects (font (size 1.27 1.27)) (justify left))
     )
@@
       (effects (font (size 1.27 1.27)) (justify left))
     )
-    (property "Value" "" (id 1) (at 53.34 176.53 0)
+    (property "Value" "100nF" (id 1) (at 53.34 176.53 0)
       (effects (font (size 1.27 1.27)) (justify left))
     )
@@
     (in_bom yes) (on_board yes) (fields_autoplaced)
     (property "Reference" "U3" (id 0) (at 227.33 100.33 0))
-    (property "Value" "" (id 1) (at 227.33 102.87 0))
+    (property "Value" "ADA4807-2ARM" (id 1) (at 227.33 102.87 0))
     (property "Footprint" "" (id 2) (at 227.33 110.49 0)
       (effects (font (size 1.27 1.27)) hide)
@@
     (in_bom yes) (on_board yes) (fields_autoplaced)
     (property "Reference" "C?" (id 0) (at 205.74 100.33 90))
-    (property "Value" "" (id 1) (at 205.74 102.87 90))
+    (property "Value" "1nF" (id 1) (at 205.74 102.87 90))
     (property "Footprint" "" (id 2) (at 209.55 106.9848 0)
       (effects (font (size 1.27 1.27)) hide)
@@
       (effects (font (size 1.27 1.27)) (justify right))
     )
-    (property "Value" "" (id 1) (at 210.82 116.84 90)
+    (property "Value" "150K" (id 1) (at 210.82 116.84 90)
       (effects (font (size 1.27 1.27)) (justify right))
     )
@@
       (effects (font (size 1.27 1.27)) (justify left))
     )
-    (property "Value" "" (id 1) (at 172.72 114.3 90)
+    (property "Value" "5.1" (id 1) (at 172.72 114.3 90)
       (effects (font (size 1.27 1.27)) (justify left))
     )
@@
       (effects (font (size 1.27 1.27)) (justify left))
     )
-    (property "Value" "" (id 1) (at 67.31 177.8 0)
-      (effects (font (size 1.27 1.27)) (justify left))
-    )
+    (property "Value" "100nF" (id 1) (at 67.31 177.8 0)
+      (effects (font (size 1.27 1.27)) (justify left))
+    )

Commit message: add ttl output; update adc voltage
Parts:
- removed R?: 68K, symbol Device:R
- removed R?: 150K, symbol Device:R
- added R?: 100K, symbol Device:R
- added R?: 10K, Resistor_SMD:R_0402_1005Metric_Pad0.72x0.64mm_HandSolder, symbol Device:R
- added RV2: R_Potentiometer_Trim, Potentiometer_SMD:Potentiometer_Bourns_3314G_Vertical, symbol Device:R_Potentiometer_Trim
- R?: value 5.1 -> 7.68; footprint (none) -> Resistor_SMD:R_0402_1005Metric_Pad0.72x0.64mm_HandSolder; Link https://www.digikey.com/en/products/detail/panasonic-electr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 -> https://www.digikey.com/en/products/detail/te-connectivity-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; Manufacturer Panasonic Electronic Components -> TE Connectivity Passive Product; Manufacturer Number ERJ-3BQF5R1V -> RP73PF1E7R68BTDF; Tolerance 1% -> 0.1%
- U4: footprint (none) -> Package_SO:MSOP-10_3x3mm_P0.5mm
Connections:
- net GNDA: now also R?.2
- net at U4.10 (VOUT): now also R?.1, RV2.2
- net at R?.1, U3.5 (+): now also R?.2, RV2.1
- net at C?.2, U3.3 (+): now also R?.1
- net +5V renamed +2V5
- net -5V renamed -2V5
Other:
- note added: "100K"
- note added: "DNP: Fixed Gain Resistor"
- note added: "High Pass Filter to remove DC offset. Fc = 15[KHz]"
- note added: "TODO: consider generating 100[KHz] sine wave with a filtered crystal output instead."
- note added: "Vout_min = 7.68/(7.68 + 100e3) * Vin = 50e-6[V]"
- note removed: "High Pass Filter to remove DC offset. Fc = 1[KHz]"
- note removed: "Vout = 5.1/(5.1 + 68e3) * Vin"

Commit message: update resistor value from 309 to 309K
Changed lines of the file:
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@@
       (effects (font (size 1.27 1.27)) hide)
     )
-    (property "Value" "" (id 1) (at 62.23 190.5 0))
+    (property "Value" "-2V5" (id 1) (at 62.23 190.5 0))
     (property "Footprint" "" (id 2) (at 62.23 186.69 0)
       (effects (font (size 1.27 1.27)) hide)
@@
       (effects (font (size 1.27 1.27)) hide)
     )
-    (property "Value" "" (id 1) (at 62.23 160.02 0))
+    (property "Value" "+2V5" (id 1) (at 62.23 160.02 0))
     (property "Footprint" "" (id 2) (at 62.23 163.83 0)
       (effects (font (size 1.27 1.27)) hide)

Commit message: add extra series termination resistors
Parts:
- C?: value 10uF -> (none)
- C? (x4): value 100nF -> (none)
- C? (x2): value 10nF -> (none)
- C?: value 1nF -> (none)
- R?: value 100K -> (none)
- R?: value 10K -> (none); footprint Resistor_SMD:R_0402_1005Metric_Pad0.72x0.64mm_HandSolder -> (none)
- R?: value 7.68 -> (none); footprint Resistor_SMD:R_0402_1005Metric_Pad0.72x0.64mm_HandSolder -> (none)
- RV2: value R_Potentiometer_Trim -> (none); footprint Potentiometer_SMD:Potentiometer_Bourns_3314G_Vertical -> (none)
- U3: value ADA4807-2ARM -> (none)
- U4: value AD9833xRM -> (none); footprint Package_SO:MSOP-10_3x3mm_P0.5mm -> (none)
- X1: value ASE-25.000MHZ-L-C-T -> (none); footprint Crystal:Crystal_SMD_Abracon_ABM8G-4Pin_3.2x2.5mm -> (none)
Changed lines of the file:
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@@
       (effects (font (size 1.27 1.27)) (justify left))
     )
-    (property "Value" "10uF" (id 1) (at 44.45 176.53 0)
+    (property "Value" "" (id 1) (at 44.45 176.53 0)
       (effects (font (size 1.27 1.27)) (justify left))
     )
@@
     (in_bom yes) (on_board yes)
     (property "Reference" "X1" (id 0) (at 99.06 91.44 0))
-    (property "Value" "ASE-25.000MHZ-L-C-T" (id 1) (at 87.63 88.9 0))
-    (property "Footprint" "Crystal:Crystal_SMD_Abracon_ABM8G-4Pin_3.2x2.5mm" (id 2) (at 120.65 106.68 0)
+    (property "Value" "" (id 1) (at 87.63 88.9 0))
+    (property "Footprint" "" (id 2) (at 120.65 106.68 0)
       (effects (font (size 1.27 1.27)) hide)
     )
@@
     (in_bom yes) (on_board yes)
     (property "Reference" "U4" (id 0) (at 124.46 81.28 0))
-    (property "Value" "AD9833xRM" (id 1) (at 144.78 81.28 0))
-    (property "Footprint" "Package_SO:MSOP-10_3x3mm_P0.5mm" (id 2) (at 135.89 107.95 0)
+    (property "Value" "" (id 1) (at 144.78 81.28 0))
+    (property "Footprint" "" (id 2) (at 135.89 107.95 0)
       (effects (font (size 1.27 1.27)) hide)
     )
@@
       (effects (font (size 1.27 1.27)) (justify left))
     )
-    (property "Value" "100nF" (id 1) (at 133.35 72.39 90)
+    (property "Value" "" (id 1) (at 133.35 72.39 90)
       (effects (font (size 1.27 1.27)) (justify left))
     )
@@
       (effects (font (size 1.27 1.27)) (justify left))
     )
-    (property "Value" "100K" (id 1) (at 173.99 102.87 0)
+    (property "Value" "" (id 1) (at 173.99 102.87 0)
       (effects (font (size 1.27 1.27)) (justify left))
     )
@@
       (effects (font (size 1.27 1.27)) (justify left))
     )
-    (property "Value" "10K" (id 1) (at 210.82 116.84 90)
-      (effects (font (size 1.27 1.27)) (justify left))
-    )
-    (property "Footprint" "Resistor_SMD:R_0402_1005Metric_Pad0.72x0.64mm_HandSolder" (id 2) (at 209.042 114.3 90)
+    (property "Value" "" (id 1) (at 210.82 116.84 90)
+      (effects (font (size 1.27 1.27)) (justify left))
+    )
+    (property "Footprint" "" (id 2) (at 209.042 114.3 90)
       (effects (font (size 1.27 1.27)) hide)
     )
@@
       (effects (font (size 1.27 1.27)) (justify left))
     )
-    (property "Value" "10nF" (id 1) (at 30.48 176.53 0)
+    (property "Value" "" (id 1) (at 30.48 176.53 0)
       (effects (font (size 1.27 1.27)) (justify left))
     )
@@
     (in_bom yes) (on_board yes) (fields_autoplaced)
     (property "Reference" "U3" (id 0) (at 191.77 100.33 0))
-    (property "Value" "ADA4807-2ARM" (id 1) (at 191.77 102.87 0))
+    (property "Value" "" (id 1) (at 191.77 102.87 0))
     (property "Footprint" "" (id 2) (at 191.77 110.49 0)
       (effects (font (size 1.27 1.27)) hide)
@@
       (effects (font (size 1.27 1.27)) (justify left))
     )
-    (property "Value" "100nF" (id 1) (at 67.31 167.64 0)
+    (property "Value" "" (id 1) (at 67.31 167.64 0)
       (effects (font (size 1.27 1.27)) (justify left))
     )
@@
       (effects (font (size 1.27 1.27)) (justify right))
     )
-    (property "Value" "10nF" (id 1) (at 157.48 85.0899 0)
+    (property "Value" "" (id 1) (at 157.48 85.0899 0)
       (effects (font (size 1.27 1.27)) (justify right))
     )
@@
       (effects (font (size 1.27 1.27)) (justify left))
     )
-    (property "Value" "ADA4807-2ARM" (id 1) (at 63.5 175.2599 0)
+    (property "Value" "" (id 1) (at 63.5 175.2599 0)
       (effects (font (size 1.27 1.27)) (justify left) hide)
     )
@@
     (in_bom yes) (on_board yes)
     (property "Reference" "RV2" (id 0) (at 161.29 101.6 90))
-    (property "Value" "R_Potentiometer_Trim" (id 1) (at 157.48 101.6 90)
-      (effects (font (size 1.27 1.27)) hide)
-    )
-    (property "Footprint" "Potentiometer_SMD:Potentiometer_Bourns_3314G_Vertical" (id 2) (at 163.83 101.6 0)
+    (property "Value" "" (id 1) (at 157.48 101.6 90)
+      (effects (font (size 1.27 1.27)) hide)
+    )
+    (property "Footprint" "" (id 2) (at 163.83 101.6 0)
       (effects (font (size 1.27 1.27)) hide)
     )
@@
       (effects (font (size 1.27 1.27)) (justify left))
     )
-    (property "Value" "100nF" (id 1) (at 53.34 176.53 0)
+    (property "Value" "" (id 1) (at 53.34 176.53 0)
       (effects (font (size 1.27 1.27)) (justify left))
     )
@@
     (in_bom yes) (on_board yes) (fields_autoplaced)
     (property "Reference" "U3" (id 0) (at 227.33 100.33 0))
-    (property "Value" "ADA4807-2ARM" (id 1) (at 227.33 102.87 0))
+    (property "Value" "" (id 1) (at 227.33 102.87 0))
     (property "Footprint" "" (id 2) (at 227.33 110.49 0)
       (effects (font (size 1.27 1.27)) hide)
@@
     (in_bom yes) (on_board yes) (fields_autoplaced)
     (property "Reference" "C?" (id 0) (at 205.74 100.33 90))
-    (property "Value" "1nF" (id 1) (at 205.74 102.87 90))
+    (property "Value" "" (id 1) (at 205.74 102.87 90))
     (property "Footprint" "" (id 2) (at 209.55 106.9848 0)
       (effects (font (size 1.27 1.27)) hide)
@@
       (effects (font (size 1.27 1.27)) (justify left))
     )
-    (property "Value" "7.68" (id 1) (at 172.72 115.57 90)
-      (effects (font (size 1.27 1.27)) (justify left))
-    )
-    (property "Footprint" "Resistor_SMD:R_0402_1005Metric_Pad0.72x0.64mm_HandSolder" (id 2) (at 170.942 113.03 90)
+    (property "Value" "" (id 1) (at 172.72 115.57 90)
+      (effects (font (size 1.27 1.27)) (justify left))
+    )
+    (property "Footprint" "" (id 2) (at 170.942 113.03 90)
       (effects (font (size 1.27 1.27)) hide)
     )
@@
       (effects (font (size 1.27 1.27)) (justify left))
     )
-    (property "Value" "100nF" (id 1) (at 67.31 177.8 0)
-      (effects (font (size 1.27 1.27)) (justify left))
-    )
+    (property "Value" "" (id 1) (at 67.31 177.8 0)
+      (effects (font (size 1.27 1.27)) (justify left))
+    )

Commit message: add driven shield
Parts:
- C?: value (none) -> 10uF; footprint (none) -> Capacitor_SMD:C_0805_2012Metric
- C? (x4): value (none) -> 100nF; footprint (none) -> Capacitor_SMD:C_0603_1608Metric_Pad1.08x0.95mm_HandSolder
- C? (x2): value (none) -> 10nF; footprint (none) -> Capacitor_SMD:C_0603_1608Metric_Pad1.08x0.95mm_HandSolder
- C?: value (none) -> 1nF
- R?: value (none) -> 100K
- R?: value (none) -> 10K; footprint (none) -> Resistor_SMD:R_0402_1005Metric_Pad0.72x0.64mm_HandSolder
- R?: value (none) -> 7.68; footprint (none) -> Resistor_SMD:R_0402_1005Metric_Pad0.72x0.64mm_HandSolder
- RV2: value (none) -> R_Potentiometer_Trim; footprint (none) -> Potentiometer_SMD:Potentiometer_Bourns_3314G_Vertical
- U3: value (none) -> ADA4807-2ARM
- U4: value (none) -> AD9833xRM; footprint (none) -> Package_SO:MSOP-10_3x3mm_P0.5mm
- X1: value (none) -> ASE-25.000MHZ-L-C-T; footprint (none) -> Crystal:Crystal_SMD_Abracon_ABM8G-4Pin_3.2x2.5mm
Changed lines of the file:
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@@
       (effects (font (size 1.27 1.27)) (justify left))
     )
-    (property "Value" "" (id 1) (at 44.45 176.53 0)
-      (effects (font (size 1.27 1.27)) (justify left))
-    )
-    (property "Footprint" "" (id 2) (at 38.4048 170.18 0)
+    (property "Value" "10uF" (id 1) (at 44.45 176.53 0)
+      (effects (font (size 1.27 1.27)) (justify left))
+    )
+    (property "Footprint" "Capacitor_SMD:C_0805_2012Metric" (id 2) (at 38.4048 170.18 0)
       (effects (font (size 1.27 1.27)) hide)
     )
@@
     (in_bom yes) (on_board yes)
     (property "Reference" "X1" (id 0) (at 99.06 91.44 0))
-    (property "Value" "" (id 1) (at 87.63 88.9 0))
-    (property "Footprint" "" (id 2) (at 120.65 106.68 0)
+    (property "Value" "ASE-25.000MHZ-L-C-T" (id 1) (at 87.63 88.9 0))
+    (property "Footprint" "Crystal:Crystal_SMD_Abracon_ABM8G-4Pin_3.2x2.5mm" (id 2) (at 120.65 106.68 0)
       (effects (font (size 1.27 1.27)) hide)
     )
@@
     (in_bom yes) (on_board yes)
     (property "Reference" "U4" (id 0) (at 124.46 81.28 0))
-    (property "Value" "" (id 1) (at 144.78 81.28 0))
-    (property "Footprint" "" (id 2) (at 135.89 107.95 0)
+    (property "Value" "AD9833xRM" (id 1) (at 144.78 81.28 0))
+    (property "Footprint" "Package_SO:MSOP-10_3x3mm_P0.5mm" (id 2) (at 135.89 107.95 0)
       (effects (font (size 1.27 1.27)) hide)
     )
@@
       (effects (font (size 1.27 1.27)) (justify left))
     )
-    (property "Value" "" (id 1) (at 133.35 72.39 90)
-      (effects (font (size 1.27 1.27)) (justify left))
-    )
-    (property "Footprint" "" (id 2) (at 129.54 73.9648 0)
+    (property "Value" "100nF" (id 1) (at 133.35 72.39 90)
+      (effects (font (size 1.27 1.27)) (justify left))
+    )
+    (property "Footprint" "Capacitor_SMD:C_0603_1608Metric_Pad1.08x0.95mm_HandSolder" (id 2) (at 129.54 73.9648 0)
       (effects (font (size 1.27 1.27)) hide)
     )
@@
       (effects (font (size 1.27 1.27)) (justify left))
     )
-    (property "Value" "" (id 1) (at 173.99 102.87 0)
+    (property "Value" "100K" (id 1) (at 173.99 102.87 0)
       (effects (font (size 1.27 1.27)) (justify left))
     )
@@
       (effects (font (size 1.27 1.27)) (justify left))
     )
-    (property "Value" "" (id 1) (at 210.82 116.84 90)
-      (effects (font (size 1.27 1.27)) (justify left))
-    )
-    (property "Footprint" "" (id 2) (at 209.042 114.3 90)
+    (property "Value" "10K" (id 1) (at 210.82 116.84 90)
+      (effects (font (size 1.27 1.27)) (justify left))
+    )
+    (property "Footprint" "Resistor_SMD:R_0402_1005Metric_Pad0.72x0.64mm_HandSolder" (id 2) (at 209.042 114.3 90)
       (effects (font (size 1.27 1.27)) hide)
     )
@@
       (effects (font (size 1.27 1.27)) (justify left))
     )
-    (property "Value" "" (id 1) (at 30.48 176.53 0)
-      (effects (font (size 1.27 1.27)) (justify left))
-    )
-    (property "Footprint" "" (id 2) (at 23.1648 170.18 0)
+    (property "Value" "10nF" (id 1) (at 30.48 176.53 0)
+      (effects (font (size 1.27 1.27)) (justify left))
+    )
+    (property "Footprint" "Capacitor_SMD:C_0603_1608Metric_Pad1.08x0.95mm_HandSolder" (id 2) (at 23.1648 170.18 0)
       (effects (font (size 1.27 1.27)) hide)
     )
@@
     (in_bom yes) (on_board yes) (fields_autoplaced)
     (property "Reference" "U3" (id 0) (at 191.77 100.33 0))
-    (property "Value" "" (id 1) (at 191.77 102.87 0))
+    (property "Value" "ADA4807-2ARM" (id 1) (at 191.77 102.87 0))
     (property "Footprint" "" (id 2) (at 191.77 110.49 0)
       (effects (font (size 1.27 1.27)) hide)
@@
       (effects (font (size 1.27 1.27)) (justify left))
     )
-    (property "Value" "" (id 1) (at 67.31 167.64 0)
-      (effects (font (size 1.27 1.27)) (justify left))
-    )
-    (property "Footprint" "" (id 2) (at 74.6252 173.99 0)
+    (property "Value" "100nF" (id 1) (at 67.31 167.64 0)
+      (effects (font (size 1.27 1.27)) (justify left))
+    )
+    (property "Footprint" "Capacitor_SMD:C_0603_1608Metric_Pad1.08x0.95mm_HandSolder" (id 2) (at 74.6252 173.99 0)
       (effects (font (size 1.27 1.27)) hide)
     )
@@
       (effects (font (size 1.27 1.27)) (justify right))
     )
-    (property "Value" "" (id 1) (at 157.48 85.0899 0)
+    (property "Value" "10nF" (id 1) (at 157.48 85.0899 0)
       (effects (font (size 1.27 1.27)) (justify right))
     )
-    (property "Footprint" "" (id 2) (at 152.7048 80.01 0)
+    (property "Footprint" "Capacitor_SMD:C_0603_1608Metric_Pad1.08x0.95mm_HandSolder" (id 2) (at 152.7048 80.01 0)
       (effects (font (size 1.27 1.27)) hide)
     )
@@
       (effects (font (size 1.27 1.27)) (justify left))
     )
-    (property "Value" "" (id 1) (at 63.5 175.2599 0)
+    (property "Value" "ADA4807-2ARM" (id 1) (at 63.5 175.2599 0)
       (effects (font (size 1.27 1.27)) (justify left) hide)
     )
@@
     (in_bom yes) (on_board yes)
     (property "Reference" "RV2" (id 0) (at 161.29 101.6 90))
-    (property "Value" "" (id 1) (at 157.48 101.6 90)
-      (effects (font (size 1.27 1.27)) hide)
-    )
-    (property "Footprint" "" (id 2) (at 163.83 101.6 0)
+    (property "Value" "R_Potentiometer_Trim" (id 1) (at 157.48 101.6 90)
+      (effects (font (size 1.27 1.27)) hide)
+    )
+    (property "Footprint" "Potentiometer_SMD:Potentiometer_Bourns_3314G_Vertical" (id 2) (at 163.83 101.6 0)
       (effects (font (size 1.27 1.27)) hide)
     )
@@
       (effects (font (size 1.27 1.27)) (justify left))
     )
-    (property "Value" "" (id 1) (at 53.34 176.53 0)
-      (effects (font (size 1.27 1.27)) (justify left))
-    )
-    (property "Footprint" "" (id 2) (at 46.0248 170.18 0)
+    (property "Value" "100nF" (id 1) (at 53.34 176.53 0)
+      (effects (font (size 1.27 1.27)) (justify left))
+    )
+    (property "Footprint" "Capacitor_SMD:C_0603_1608Metric_Pad1.08x0.95mm_HandSolder" (id 2) (at 46.0248 170.18 0)
       (effects (font (size 1.27 1.27)) hide)
     )
@@
     (in_bom yes) (on_board yes) (fields_autoplaced)
     (property "Reference" "U3" (id 0) (at 227.33 100.33 0))
-    (property "Value" "" (id 1) (at 227.33 102.87 0))
+    (property "Value" "ADA4807-2ARM" (id 1) (at 227.33 102.87 0))
     (property "Footprint" "" (id 2) (at 227.33 110.49 0)
       (effects (font (size 1.27 1.27)) hide)
@@
     (in_bom yes) (on_board yes) (fields_autoplaced)
     (property "Reference" "C?" (id 0) (at 205.74 100.33 90))
-    (property "Value" "" (id 1) (at 205.74 102.87 90))
+    (property "Value" "1nF" (id 1) (at 205.74 102.87 90))
     (property "Footprint" "" (id 2) (at 209.55 106.9848 0)
       (effects (font (size 1.27 1.27)) hide)
@@
       (effects (font (size 1.27 1.27)) (justify left))
     )
-    (property "Value" "" (id 1) (at 172.72 115.57 90)
-      (effects (font (size 1.27 1.27)) (justify left))
-    )
-    (property "Footprint" "" (id 2) (at 170.942 113.03 90)
+    (property "Value" "7.68" (id 1) (at 172.72 115.57 90)
+      (effects (font (size 1.27 1.27)) (justify left))
+    )
+    (property "Footprint" "Resistor_SMD:R_0402_1005Metric_Pad0.72x0.64mm_HandSolder" (id 2) (at 170.942 113.03 90)
       (effects (font (size 1.27 1.27)) hide)
     )
@@
       (effects (font (size 1.27 1.27)) (justify left))
     )
-    (property "Value" "" (id 1) (at 67.31 177.8 0)
-      (effects (font (size 1.27 1.27)) (justify left))
-    )
-    (property "Footprint" "" (id 2) (at 74.6252 184.15 0)
-      (effects (font (size 1.27 1.27)) hide)
-    )
+    (property "Value" "100nF" (id 1) (at 67.31 177.8 0)
+      (effects (font (size 1.27 1.27)) (justify left))
+    )
+    (property "Footprint" "Capacitor_SMD:C_0603_1608Metric_Pad1.08x0.95mm_HandSolder" (id 2) (at 74.6252 184.15 0)
+      (effects (font (size 1.27 1.27)) hide)
+    )
