File: hardware/board/harp_lick_detector_capactive/sine_wave_source.kicad_sch (KiCad schematic)
At the start: 18 parts, among them U10 LTC6263, U7 AD9833xRM, X2 ASE-25.000MHZ-L-C-T

Commit message: complete bom assignment
Parts:
- C25, C31: value 10nF -> (none); footprint Capacitor_SMD:C_0603_1608Metric_Pad1.08x0.95mm_HandSolder -> (none)
- C26: value 10uF -> (none); footprint Capacitor_SMD:C_0805_2012Metric -> (none)
- C27, C28, C29, C30: value 100nF -> (none); footprint Capacitor_SMD:C_0603_1608Metric_Pad1.08x0.95mm_HandSolder -> (none)
- C41, C42: value 160pF -> (none); footprint Capacitor_SMD:C_0402_1005Metric_Pad0.74x0.62mm_HandSolder -> (none)
- R18: value 100K -> (none); Link (none) -> https://www.digikey.com/en/products/detail/yageo/RC0402FR-1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; Manufacturer (none) -> Yageo; Manufacturer Number (none) -> RC0402FR-13100KL; Tolerance (none) -> 1%
- R19: value 7.68 -> (none); footprint Resistor_SMD:R_0402_1005Metric_Pad0.72x0.64mm_HandSolder -> (none)
- R34: value 99K2 -> (none); Link (none) -> https://www.digikey.com/en/products/detail/koa-speer-electr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; Manufacturer (none) -> KOA Spear Electronics, Inc.; Manufacturer Number (none) -> RN73H1JTTD9882B25; Notes (none) -> ideally would be 99K2; Tolerance (none) -> 0.1%
- R35: value 501 -> (none); Link (none) -> https://www.digikey.com/en/products/detail/yageo/RT0603BRC0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; Manufacturer (none) -> Yageo; Manufacturer Number (none) -> RT0603BRC07500RL; Notes (none) -> Ideally would be 501; Tolerance (none) -> 0.1%
- R36: value 198K -> (none); Link (none) -> https://www.digikey.com/en/products/detail/yageo/RT0603BRD0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; Manufacturer (none) -> Yageo; Manufacturer Number (none) -> RT0603BRD07200KL; Notes (none) -> ideally would be 198K; Tolerance (none) -> 0.1%
- RV2: value R_Potentiometer_Trim -> (none); footprint Potentiometer_SMD:Potentiometer_Bourns_3314G_Vertical -> (none)
- U10: value LTC6263 -> (none); footprint Package_SO:MSOP-16_3x4mm_P0.5mm -> (none)
- U7: value AD9833xRM -> (none); footprint Package_SO:MSOP-10_3x3mm_P0.5mm -> (none)
- X2: value ASE-25.000MHZ-L-C-T -> (none); footprint Crystal:Crystal_SMD_Abracon_ABM8G-4Pin_3.2x2.5mm -> (none)

Commit message: loosely place components
Parts:
- C27, C28, C29, C30: Link https://www.digikey.com/en/products/detail/samsung-electro-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 -> https://www.digikey.com/en/products/detail/walsin-technolog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; Manufacturer Samsung Electro-Mechanics -> Walson Technology Corporation; Manufacturer Number CL10B104KB8NNWC -> 0402B104K160CT; Rated Voltage 50V -> 16V
Changed lines of the file:
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@@
       (effects (font (size 1.27 1.27)) hide)
     )
-    (property "Datasheet" "https://media.digikey.com/pdf/Data%20Sheets/Samsung%20PDFs/CL10B104KB8NNWC_Spec.pdf" (id 3) (at 125.73 74.93 0)
-      (effects (font (size 1.27 1.27)) hide)
-    )
-    (property "Link" "https://www.digikey.com/en/products/detail/samsung-electro-mechanics/CL10B104KB8NNWC/3887593" (id 4) (at 125.73 74.93 0)
-      (effects (font (size 1.27 1.27)) hide)
-    )
-    (property "Manufacturer" "Samsung Electro-Mechanics" (id 5) (at 125.73 74.93 0)
-      (effects (font (size 1.27 1.27)) hide)
-    )
-    (property "Manufacturer Number" "CL10B104KB8NNWC" (id 6) (at 125.73 74.93 0)
-      (effects (font (size 1.27 1.27)) hide)
-    )
-    (property "Rated Voltage" "50V" (id 7) (at 125.73 74.93 0)
+    (property "Datasheet" "http://www.passivecomponent.com/wp-content/uploads/datasheet/WTC_MLCC_General_Purpose.pdf" (id 3) (at 125.73 74.93 0)
+      (effects (font (size 1.27 1.27)) hide)
+    )
+    (property "Link" "https://www.digikey.com/en/products/detail/walsin-technology-corporation/0402B104K160CT/6707534" (id 4) (at 125.73 74.93 0)
+      (effects (font (size 1.27 1.27)) hide)
+    )
+    (property "Manufacturer" "Walson Technology Corporation" (id 5) (at 125.73 74.93 0)
+      (effects (font (size 1.27 1.27)) hide)
+    )
+    (property "Manufacturer Number" "0402B104K160CT" (id 6) (at 125.73 74.93 0)
+      (effects (font (size 1.27 1.27)) hide)
+    )
+    (property "Rated Voltage" "16V" (id 7) (at 125.73 74.93 0)
       (effects (font (size 1.27 1.27)) hide)
     )
@@
       (effects (font (size 1.27 1.27)) hide)
     )
-    (property "Datasheet" "https://media.digikey.com/pdf/Data%20Sheets/Samsung%20PDFs/CL10B104KB8NNWC_Spec.pdf" (id 3) (at 80.01 168.91 0)
-      (effects (font (size 1.27 1.27)) hide)
-    )
-    (property "Link" "https://www.digikey.com/en/products/detail/samsung-electro-mechanics/CL10B104KB8NNWC/3887593" (id 4) (at 80.01 168.91 0)
-      (effects (font (size 1.27 1.27)) hide)
-    )
-    (property "Manufacturer" "Samsung Electro-Mechanics" (id 5) (at 80.01 168.91 0)
-      (effects (font (size 1.27 1.27)) hide)
-    )
-    (property "Manufacturer Number" "CL10B104KB8NNWC" (id 6) (at 80.01 168.91 0)
-      (effects (font (size 1.27 1.27)) hide)
-    )
-    (property "Rated Voltage" "50V" (id 7) (at 80.01 168.91 0)
+    (property "Datasheet" "http://www.passivecomponent.com/wp-content/uploads/datasheet/WTC_MLCC_General_Purpose.pdf" (id 3) (at 80.01 168.91 0)
+      (effects (font (size 1.27 1.27)) hide)
+    )
+    (property "Link" "https://www.digikey.com/en/products/detail/walsin-technology-corporation/0402B104K160CT/6707534" (id 4) (at 80.01 168.91 0)
+      (effects (font (size 1.27 1.27)) hide)
+    )
+    (property "Manufacturer" "Walson Technology Corporation" (id 5) (at 80.01 168.91 0)
+      (effects (font (size 1.27 1.27)) hide)
+    )
+    (property "Manufacturer Number" "0402B104K160CT" (id 6) (at 80.01 168.91 0)
+      (effects (font (size 1.27 1.27)) hide)
+    )
+    (property "Rated Voltage" "16V" (id 7) (at 80.01 168.91 0)
       (effects (font (size 1.27 1.27)) hide)
     )
@@
       (effects (font (size 1.27 1.27)) hide)
     )
-    (property "Datasheet" "https://media.digikey.com/pdf/Data%20Sheets/Samsung%20PDFs/CL10B104KB8NNWC_Spec.pdf" (id 3) (at 46.99 173.99 0)
-      (effects (font (size 1.27 1.27)) hide)
-    )
-    (property "Link" "https://www.digikey.com/en/products/detail/samsung-electro-mechanics/CL10B104KB8NNWC/3887593" (id 4) (at 46.99 173.99 0)
-      (effects (font (size 1.27 1.27)) hide)
-    )
-    (property "Manufacturer" "Samsung Electro-Mechanics" (id 5) (at 46.99 173.99 0)
-      (effects (font (size 1.27 1.27)) hide)
-    )
-    (property "Manufacturer Number" "CL10B104KB8NNWC" (id 6) (at 46.99 173.99 0)
-      (effects (font (size 1.27 1.27)) hide)
-    )
-    (property "Rated Voltage" "50V" (id 7) (at 46.99 173.99 0)
+    (property "Datasheet" "http://www.passivecomponent.com/wp-content/uploads/datasheet/WTC_MLCC_General_Purpose.pdf" (id 3) (at 46.99 173.99 0)
+      (effects (font (size 1.27 1.27)) hide)
+    )
+    (property "Link" "https://www.digikey.com/en/products/detail/walsin-technology-corporation/0402B104K160CT/6707534" (id 4) (at 46.99 173.99 0)
+      (effects (font (size 1.27 1.27)) hide)
+    )
+    (property "Manufacturer" "Walson Technology Corporation" (id 5) (at 46.99 173.99 0)
+      (effects (font (size 1.27 1.27)) hide)
+    )
+    (property "Manufacturer Number" "0402B104K160CT" (id 6) (at 46.99 173.99 0)
+      (effects (font (size 1.27 1.27)) hide)
+    )
+    (property "Rated Voltage" "16V" (id 7) (at 46.99 173.99 0)
       (effects (font (size 1.27 1.27)) hide)
     )
@@
       (effects (font (size 1.27 1.27)) hide)
     )
-    (property "Datasheet" "https://media.digikey.com/pdf/Data%20Sheets/Samsung%20PDFs/CL10B104KB8NNWC_Spec.pdf" (id 3) (at 80.01 179.07 0)
-      (effects (font (size 1.27 1.27)) hide)
-    )
-    (property "Link" "https://www.digikey.com/en/products/detail/samsung-electro-mechanics/CL10B104KB8NNWC/3887593" (id 4) (at 80.01 179.07 0)
-      (effects (font (size 1.27 1.27)) hide)
-    )
-    (property "Manufacturer" "Samsung Electro-Mechanics" (id 5) (at 80.01 179.07 0)
-      (effects (font (size 1.27 1.27)) hide)
-    )
-    (property "Manufacturer Number" "CL10B104KB8NNWC" (id 6) (at 80.01 179.07 0)
-      (effects (font (size 1.27 1.27)) hide)
-    )
-    (property "Rated Voltage" "50V" (id 7) (at 80.01 179.07 0)
-      (effects (font (size 1.27 1.27)) hide)
-    )
+    (property "Datasheet" "http://www.passivecomponent.com/wp-content/uploads/datasheet/WTC_MLCC_General_Purpose.pdf" (id 3) (at 80.01 179.07 0)
+      (effects (font (size 1.27 1.27)) hide)
+    )
+    (property "Link" "https://www.digikey.com/en/products/detail/walsin-technology-corporation/0402B104K160CT/6707534" (id 4) (at 80.01 179.07 0)
+      (effects (font (size 1.27 1.27)) hide)
+    )
+    (property "Manufacturer" "Walson Technology Corporation" (id 5) (at 80.01 179.07 0)
+      (effects (font (size 1.27 1.27)) hide)
+    )
+    (property "Manufacturer Number" "0402B104K160CT" (id 6) (at 80.01 179.07 0)
+      (effects (font (size 1.27 1.27)) hide)
+    )
+    (property "Rated Voltage" "16V" (id 7) (at 80.01 179.07 0)
+      (effects (font (size 1.27 1.27)) hide)
+    )

Commit message: change usb connector; more layout
Parts:
- C25, C31: value (none) -> 10nF; footprint (none) -> Capacitor_SMD:C_0603_1608Metric_Pad1.08x0.95mm_HandSolder
- C26: value (none) -> 10uF; footprint (none) -> Capacitor_SMD:C_0805_2012Metric
- C27, C28, C29, C30: value (none) -> 100nF; footprint (none) -> Capacitor_SMD:C_0402_1005Metric_Pad0.74x0.62mm_HandSolder
- C41, C42: value (none) -> 160pF; footprint (none) -> Capacitor_SMD:C_0402_1005Metric_Pad0.74x0.62mm_HandSolder
- R18: value (none) -> 100K; footprint (none) -> Resistor_SMD:R_0402_1005Metric_Pad0.72x0.64mm_HandSolder
- R19: value (none) -> 7.68; footprint (none) -> Resistor_SMD:R_0402_1005Metric_Pad0.72x0.64mm_HandSolder
- R34: value (none) -> 98K8; footprint (none) -> Resistor_SMD:R_0603_1608Metric_Pad0.98x0.95mm_HandSolder
- R35: value (none) -> 501; footprint (none) -> Resistor_SMD:R_0603_1608Metric_Pad0.98x0.95mm_HandSolder
- R36: value (none) -> 200K; footprint (none) -> Resistor_SMD:R_0603_1608Metric_Pad0.98x0.95mm_HandSolder
- RV2: value (none) -> R_Potentiometer_Trim; footprint (none) -> Potentiometer_SMD:Potentiometer_Bourns_3314G_Vertical
- U10: value (none) -> LTC6263; footprint (none) -> Package_SO:MSOP-16_3x4mm_P0.5mm
- U7: value (none) -> AD9833xRM; footprint (none) -> Package_SO:MSOP-10_3x3mm_P0.5mm
- X2: value (none) -> ASE-25.000MHZ-L-C-T; footprint (none) -> Crystal:Crystal_SMD_Abracon_ABM8G-4Pin_3.2x2.5mm

Commit message: add analog front end test board
Parts:
- R36: value 200K -> 198K; footprint Resistor_SMD:R_0603_1608Metric_Pad0.98x0.95mm_HandSolder -> Resistor_SMD:R_0402_1005Metric_Pad0.72x0.64mm_HandSolder; Link https://www.digikey.com/en/products/detail/yageo/RT0603BRD0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 -> https://www.mouser.com/ProductDetail/YAGEO/RT0603BRD07198KL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; Manufacturer Number RT0603BRD07200KL -> RT0603BRD07198KL
Changed lines of the file:
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@@
     (in_bom yes) (on_board yes)
     (property "Reference" "R36" (id 0) (at 226.06 101.6 0))
-    (property "Value" "200K" (id 1) (at 223.52 105.41 90))
-    (property "Footprint" "Resistor_SMD:R_0603_1608Metric_Pad0.98x0.95mm_HandSolder" (id 2) (at 225.298 105.41 90)
+    (property "Value" "198K" (id 1) (at 223.52 105.41 90))
+    (property "Footprint" "Resistor_SMD:R_0402_1005Metric_Pad0.72x0.64mm_HandSolder" (id 2) (at 225.298 105.41 90)
       (effects (font (size 1.27 1.27)) hide)
     )
-    (property "Datasheet" "https://www.yageo.com/upload/media/product/productsearch/datasheet/rchip/PYu-RT_1-to-0.01_RoHS_L_15.pdf" (id 3) (at 223.52 105.41 0)
+    (property "Datasheet" "https://www.mouser.com/datasheet/2/447/PYu_RT_1_to_0_01_RoHS_L_12-3003070.pdf" (id 3) (at 223.52 105.41 0)
       (effects (font (size 1.27 1.27)) hide)
     )
-    (property "Link" "https://www.digikey.com/en/products/detail/yageo/RT0603BRD07200KL/1072345" (id 4) (at 223.52 105.41 0)
+    (property "Link" "https://www.mouser.com/ProductDetail/YAGEO/RT0603BRD07198KL?qs=bQfrgN9vNvxjjoB%252BIKRwPQ%3D%3D" (id 4) (at 223.52 105.41 0)
       (effects (font (size 1.27 1.27)) hide)
     )
@@
       (effects (font (size 1.27 1.27)) hide)
     )
-    (property "Manufacturer Number" "RT0603BRD07200KL" (id 6) (at 223.52 105.41 0)
+    (property "Manufacturer Number" "RT0603BRD07198KL" (id 6) (at 223.52 105.41 0)
       (effects (font (size 1.27 1.27)) hide)
     )

Commit message: update bandpass filter; plan pico shield version
Connections:
- net GND is gone; now on net GNDA: U7.4 (DGND)
Other:
- note added: "Datasheet: "Digital and analog ground planes should be joined in one place only." If the AD9833 is the only device requiring split grounds, join the AD9833 AGND and DGND pins."
- note removed: "Datasheet: "Digital and analog ground planes should be joined in one place only.""
Changed lines of the file:
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@@
   (junction (at 68.58 163.83) (diameter 0) (color 0 0 0 0)
+  )
+  (junction (at 138.43 106.68) (diameter 0) (color 0 0 0 0)
   )
   (junction (at 200.66 113.03) (diameter 0) (color 0 0 0 0)
@@
     (stroke (width 0) (type default) (color 0 0 0 0))
   )
-  (wire (pts (xy 133.35 105.41) (xy 133.35 107.95))
+  (wire (pts (xy 133.35 105.41) (xy 133.35 106.68))
     (stroke (width 0) (type default) (color 0 0 0 0))
   )
@@
     (stroke (width 0) (type default) (color 0 0 0 0))
   )
+  (wire (pts (xy 133.35 106.68) (xy 138.43 106.68))
+    (stroke (width 0) (type default) (color 0 0 0 0))
+  )
   (wire (pts (xy 184.15 113.03) (xy 182.88 113.03))
     (stroke (width 0) (type default) (color 0 0 0 0))
@@
     (stroke (width 0) (type default) (color 0 0 0 0))
   )
-  (wire (pts (xy 138.43 105.41) (xy 138.43 107.95))
+  (wire (pts (xy 138.43 105.41) (xy 138.43 106.68))
     (stroke (width 0) (type default) (color 0 0 0 0))
   )
@@
   )
   (wire (pts (xy 172.72 107.95) (xy 172.72 109.22))
+    (stroke (width 0) (type default) (color 0 0 0 0))
+  )
+  (wire (pts (xy 138.43 106.68) (xy 138.43 107.95))
     (stroke (width 0) (type default) (color 0 0 0 0))
   )
@@
     (effects (font (size 1.27 1.27)) (justify left bottom))
   )
-  (text "Datasheet: \"Digital and analog ground planes should be\njoined in one place only.\""
+  (text "Datasheet: \"Digital and analog ground planes should be\njoined in one place only.\" If the AD9833 is the only \ndevice requiring split grounds, join the AD9833\nAGND and DGND pins."
     (at 120.65 142.24 0)
     (effects (font (size 1.27 1.27)) (justify left bottom))
@@
     (pin "2")
   )
-  (symbol (lib_id "power:GND") (at 133.35 107.95 0) (unit 1)
-    (in_bom yes) (on_board yes)
-    (property "Reference" "#PWR0146" (id 0) (at 133.35 114.3 0)
-      (effects (font (size 1.27 1.27)) hide)
-    )
-    (property "Value" "GND" (id 1) (at 134.62 111.76 0)
-      (effects (font (size 1.27 1.27)) (justify right))
-    )
-    (property "Footprint" "" (id 2) (at 133.35 107.95 0)
-      (effects (font (size 1.27 1.27)) hide)
-    )
-    (property "Datasheet" "" (id 3) (at 133.35 107.95 0)
-      (effects (font (size 1.27 1.27)) hide)
-    )
-    (pin "1")
-  )
   (symbol (lib_id "Device:C") (at 153.67 83.82 180) (unit 1)
