File: hardware/board/harp_lick_detector_capactive/ttl_output.kicad_sch (KiCad schematic)
At the start: 8 parts

Commit message: update resistor value from 309 to 309K
Changed lines of the file:
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@@
       (effects (font (size 1.27 1.27)) hide)
     )
-    (property "Value" "" (id 1) (at 24.13 156.21 0))
+    (property "Value" "+5V" (id 1) (at 24.13 156.21 0))
     (property "Footprint" "" (id 2) (at 24.13 160.02 0)
       (effects (font (size 1.27 1.27)) hide)
@@
       (effects (font (size 1.27 1.27)) hide)
     )
-    (property "Value" "" (id 1) (at 45.72 165.1 0))
+    (property "Value" "+5V" (id 1) (at 45.72 165.1 0))
     (property "Footprint" "" (id 2) (at 45.72 168.91 0)
       (effects (font (size 1.27 1.27)) hide)

Commit message: document stray capacitances
Parts:
- gave numbers to parts that had none: 4
Changed lines of the file:
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@@
   (symbol (lib_id "power:GND") (at 171.45 97.79 0) (unit 1)
     (in_bom yes) (on_board yes) (fields_autoplaced)
-    (property "Reference" "#PWR?" (id 0) (at 171.45 104.14 0)
+    (property "Reference" "#PWR0192" (id 0) (at 171.45 104.14 0)
       (effects (font (size 1.27 1.27)) hide)
     )
@@
   (symbol (lib_id "power:+5V") (at 24.13 160.02 0) (unit 1)
     (in_bom yes) (on_board yes)
-    (property "Reference" "#PWR?" (id 0) (at 24.13 163.83 0)
+    (property "Reference" "#PWR0190" (id 0) (at 24.13 163.83 0)
       (effects (font (size 1.27 1.27)) hide)
     )
@@
   (symbol (lib_id "74xx:74HC04") (at 144.78 91.44 0) (unit 3)
     (in_bom yes) (on_board yes)
-    (property "Reference" "U?" (id 0) (at 147.32 85.09 0))
+    (property "Reference" "U11" (id 0) (at 147.32 85.09 0))
     (property "Value" "74HC04" (id 1) (at 147.32 87.63 0))
     (property "Footprint" "" (id 2) (at 144.78 91.44 0)
@@
   (symbol (lib_id "Connector:Conn_Coaxial") (at 171.45 91.44 0) (unit 1)
     (in_bom yes) (on_board yes) (fields_autoplaced)
-    (property "Reference" "J?" (id 0) (at 173.99 90.4631 0)
+    (property "Reference" "J9" (id 0) (at 173.99 90.4631 0)
       (effects (font (size 1.27 1.27)) (justify left))
     )
@@
   (symbol (lib_id "74xx:74HC04") (at 144.78 102.87 0) (unit 4)
     (in_bom yes) (on_board yes)
-    (property "Reference" "U?" (id 0) (at 146.05 96.52 0))
+    (property "Reference" "U11" (id 0) (at 146.05 96.52 0))
     (property "Value" "74HC04" (id 1) (at 147.32 99.06 0))
     (property "Footprint" "" (id 2) (at 144.78 102.87 0)
@@
   (symbol (lib_id "74xx:74HC04") (at 144.78 81.28 0) (unit 2)
     (in_bom yes) (on_board yes)
-    (property "Reference" "U?" (id 0) (at 147.32 74.93 0))
+    (property "Reference" "U11" (id 0) (at 147.32 74.93 0))
     (property "Value" "74HC04" (id 1) (at 147.32 77.47 0))
     (property "Footprint" "" (id 2) (at 144.78 81.28 0)
@@
   (symbol (lib_id "power:GND") (at 24.13 187.96 0) (unit 1)
     (in_bom yes) (on_board yes) (fields_autoplaced)
-    (property "Reference" "#PWR?" (id 0) (at 24.13 194.31 0)
+    (property "Reference" "#PWR0191" (id 0) (at 24.13 194.31 0)
       (effects (font (size 1.27 1.27)) hide)
     )
@@
   (symbol (lib_id "power:GND") (at 45.72 179.07 0) (unit 1)
     (in_bom yes) (on_board yes) (fields_autoplaced)
-    (property "Reference" "#PWR?" (id 0) (at 45.72 185.42 0)
+    (property "Reference" "#PWR0188" (id 0) (at 45.72 185.42 0)
       (effects (font (size 1.27 1.27)) hide)
     )
@@
   (symbol (lib_id "Device:C") (at 45.72 173.99 0) (unit 1)
     (in_bom yes) (on_board yes)
-    (property "Reference" "C?" (id 0) (at 46.99 171.45 0)
+    (property "Reference" "C40" (id 0) (at 46.99 171.45 0)
       (effects (font (size 1.27 1.27)) (justify left))
     )
@@
   (symbol (lib_id "power:+5V") (at 45.72 168.91 0) (unit 1)
     (in_bom yes) (on_board yes)
-    (property "Reference" "#PWR?" (id 0) (at 45.72 172.72 0)
+    (property "Reference" "#PWR0189" (id 0) (at 45.72 172.72 0)
       (effects (font (size 1.27 1.27)) hide)
     )
@@
   (symbol (lib_id "74xx:74HC04") (at 24.13 173.99 0) (unit 7)
     (in_bom yes) (on_board yes) (fields_autoplaced)
-    (property "Reference" "U?" (id 0) (at 30.48 172.7199 0)
+    (property "Reference" "U11" (id 0) (at 30.48 172.7199 0)
       (effects (font (size 1.27 1.27)) (justify left))
     )
@@
   (symbol (lib_id "Device:R") (at 160.02 91.44 90) (unit 1)
     (in_bom yes) (on_board yes)
-    (property "Reference" "R?" (id 0) (at 158.75 88.9 90))
+    (property "Reference" "R33" (id 0) (at 158.75 88.9 90))
     (property "Value" "47" (id 1) (at 160.02 91.44 90))
     (property "Footprint" "" (id 2) (at 160.02 93.218 90)
@@
   (symbol (lib_id "74xx:74HC04") (at 125.73 91.44 0) (unit 1)
     (in_bom yes) (on_board yes) (fields_autoplaced)
-    (property "Reference" "U?" (id 0) (at 125.73 82.55 0))
+    (property "Reference" "U11" (id 0) (at 125.73 82.55 0))
     (property "Value" "74HC04" (id 1) (at 125.73 85.09 0))
     (property "Footprint" "" (id 2) (at 125.73 91.44 0)

Commit message: complete bom assignment
Parts:
- removed R33: 47, symbol Device:R
- removed U11: 74HC04, symbol 74xx:74HC04
- added R24, R25: (no value), symbol Device:R
- added U11: (no value), symbol 74xx:74AHC04
- C40: value 10uF -> (none); footprint Capacitor_SMD:C_0805_2012Metric -> (none)
- J9: value Conn_Coaxial -> (none)
Connections:
- net +5V: now also U11.14 (VCC)
- net GND: now also U11.7 (GND)
- net IN: now also U11.3
- net at J9.1 (In): now also R24.2, R25.2
- new net: R24.1, R25.1, U11.10, U11.12, U11.8
- new net: U11.11, U11.13, U11.4, U11.9
- no-connect marks 0 -> 4

Commit message: change usb connector; more layout
Parts:
- C40: value (none) -> 10uF; footprint (none) -> Capacitor_SMD:C_0805_2012Metric
- J9: value (none) -> Conn_Coaxial; footprint (none) -> machine_agency_components:conn_bnc_receptacle_50ohm
- R24, R25: value (none) -> 100; footprint (none) -> Resistor_SMD:R_0603_1608Metric_Pad0.98x0.95mm_HandSolder
- U11: value (none) -> CD74AC04; footprint (none) -> Package_SO:SOIC-14_3.9x8.7mm_P1.27mm
Changed lines of the file:
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@@
     (in_bom yes) (on_board yes)
     (property "Reference" "U11" (id 0) (at 148.59 93.98 0))
-    (property "Value" "" (id 1) (at 148.59 87.63 0))
-    (property "Footprint" "" (id 2) (at 144.78 91.44 0)
+    (property "Value" "CD74AC04" (id 1) (at 148.59 87.63 0))
+    (property "Footprint" "Package_SO:SOIC-14_3.9x8.7mm_P1.27mm" (id 2) (at 144.78 91.44 0)
       (effects (font (size 1.27 1.27)) hide)
     )
@@
     (in_bom yes) (on_board yes)
     (property "Reference" "R25" (id 0) (at 161.29 96.52 90))
-    (property "Value" "" (id 1) (at 161.29 93.98 90))
-    (property "Footprint" "" (id 2) (at 161.29 95.758 90)
+    (property "Value" "100" (id 1) (at 161.29 93.98 90))
+    (property "Footprint" "Resistor_SMD:R_0603_1608Metric_Pad0.98x0.95mm_HandSolder" (id 2) (at 161.29 95.758 90)
       (effects (font (size 1.27 1.27)) hide)
     )
@@
       (effects (font (size 1.27 1.27)) (justify left))
     )
-    (property "Value" "" (id 1) (at 173.99 93.0031 0)
-      (effects (font (size 1.27 1.27)) (justify left))
-    )
-    (property "Footprint" "" (id 2) (at 171.45 91.44 0)
+    (property "Value" "Conn_Coaxial" (id 1) (at 173.99 93.0031 0)
+      (effects (font (size 1.27 1.27)) (justify left))
+    )
+    (property "Footprint" "machine_agency_components:conn_bnc_receptacle_50ohm" (id 2) (at 171.45 91.44 0)
       (effects (font (size 1.27 1.27)) hide)
     )
@@
       (effects (font (size 1.27 1.27)) (justify left))
     )
-    (property "Value" "" (id 1) (at 30.48 175.2599 0)
-      (effects (font (size 1.27 1.27)) (justify left))
-    )
-    (property "Footprint" "" (id 2) (at 24.13 173.99 0)
+    (property "Value" "CD74AC04" (id 1) (at 30.48 175.2599 0)
+      (effects (font (size 1.27 1.27)) (justify left))
+    )
+    (property "Footprint" "Package_SO:SOIC-14_3.9x8.7mm_P1.27mm" (id 2) (at 24.13 173.99 0)
       (effects (font (size 1.27 1.27)) hide)
     )
@@
     (in_bom yes) (on_board yes)
     (property "Reference" "U11" (id 0) (at 148.59 135.89 0))
-    (property "Value" "" (id 1) (at 148.59 129.54 0))
-    (property "Footprint" "" (id 2) (at 144.78 133.35 0)
+    (property "Value" "CD74AC04" (id 1) (at 148.59 129.54 0))
+    (property "Footprint" "Package_SO:SOIC-14_3.9x8.7mm_P1.27mm" (id 2) (at 144.78 133.35 0)
       (effects (font (size 1.27 1.27)) hide)
     )
@@
     (in_bom yes) (on_board yes)
     (property "Reference" "R24" (id 0) (at 161.29 86.36 90))
-    (property "Value" "" (id 1) (at 161.29 88.9 90))
-    (property "Footprint" "" (id 2) (at 161.29 90.678 90)
+    (property "Value" "100" (id 1) (at 161.29 88.9 90))
+    (property "Footprint" "Resistor_SMD:R_0603_1608Metric_Pad0.98x0.95mm_HandSolder" (id 2) (at 161.29 90.678 90)
       (effects (font (size 1.27 1.27)) hide)
     )
@@
       (effects (font (size 1.27 1.27)) (justify left))
     )
-    (property "Value" "" (id 1) (at 46.99 176.53 0)
-      (effects (font (size 1.27 1.27)) (justify left))
-    )
-    (property "Footprint" "" (id 2) (at 46.6852 177.8 0)
+    (property "Value" "10uF" (id 1) (at 46.99 176.53 0)
+      (effects (font (size 1.27 1.27)) (justify left))
+    )
+    (property "Footprint" "Capacitor_SMD:C_0805_2012Metric" (id 2) (at 46.6852 177.8 0)
       (effects (font (size 1.27 1.27)) hide)
     )
@@
     (in_bom yes) (on_board yes)
     (property "Reference" "U11" (id 0) (at 148.59 83.82 0))
-    (property "Value" "" (id 1) (at 148.59 77.47 0))
-    (property "Footprint" "" (id 2) (at 144.78 81.28 0)
+    (property "Value" "CD74AC04" (id 1) (at 148.59 77.47 0))
+    (property "Footprint" "Package_SO:SOIC-14_3.9x8.7mm_P1.27mm" (id 2) (at 144.78 81.28 0)
       (effects (font (size 1.27 1.27)) hide)
     )
@@
     (in_bom yes) (on_board yes)
     (property "Reference" "U11" (id 0) (at 128.27 93.98 0))
-    (property "Value" "" (id 1) (at 128.27 87.63 0))
-    (property "Footprint" "" (id 2) (at 124.46 91.44 0)
+    (property "Value" "CD74AC04" (id 1) (at 128.27 87.63 0))
+    (property "Footprint" "Package_SO:SOIC-14_3.9x8.7mm_P1.27mm" (id 2) (at 124.46 91.44 0)
       (effects (font (size 1.27 1.27)) hide)
     )
@@
     (in_bom yes) (on_board yes)
     (property "Reference" "U11" (id 0) (at 148.59 149.86 0))
-    (property "Value" "" (id 1) (at 148.59 143.51 0))
-    (property "Footprint" "" (id 2) (at 144.78 147.32 0)
+    (property "Value" "CD74AC04" (id 1) (at 148.59 143.51 0))
+    (property "Footprint" "Package_SO:SOIC-14_3.9x8.7mm_P1.27mm" (id 2) (at 144.78 147.32 0)
       (effects (font (size 1.27 1.27)) hide)
     )
@@
     (in_bom yes) (on_board yes)
     (property "Reference" "U11" (id 0) (at 148.59 105.41 0))
-    (property "Value" "" (id 1) (at 148.59 99.06 0))
-    (property "Footprint" "" (id 2) (at 144.78 102.87 0)
-      (effects (font (size 1.27 1.27)) hide)
-    )
+    (property "Value" "CD74AC04" (id 1) (at 148.59 99.06 0))
+    (property "Footprint" "Package_SO:SOIC-14_3.9x8.7mm_P1.27mm" (id 2) (at 144.78 102.87 0)
+      (effects (font (size 1.27 1.27)) hide)
+    )
