File: hardware/board/harp_lick_detector_capactive/isolated_usb_rp2040.kicad_sch (KiCad schematic)
At the start: 47 parts, among them J2 Conn_01x03_Male, J4 AudioJack3, J5 USB_C_Receptacle_USB2.0, SW1 SW_Push, U2 TPD2EUSB30, U3 ADUM4160, U4 RP2040, U5 W25Q128JVS, X1 ECS-TXO-2016

Commit message: remove hand-soldering footprints
Parts:
- C1, C12, C13, C14, C15, C16, C17, C18, C19, C2, C3, C37, C5, C6, C7: footprint Capacitor_SMD:C_0402_1005Metric_Pad0.74x0.62mm_HandSolder -> Capacitor_SMD:C_0402_1005Metric
- J2: Alternate (none) -> n/a; Link (none) -> n/a; Manufacturer (none) -> n/a; Manufacturer Number (none) -> n/a
- R10, R11, R4, R5, R6, R7: footprint Resistor_SMD:R_0402_1005Metric_Pad0.72x0.64mm_HandSolder -> Resistor_SMD:R_0402_1005Metric
Changed lines of the file:
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@@
       (effects (font (size 1.27 1.27)))
     )
-    (property "Footprint" "Resistor_SMD:R_0402_1005Metric_Pad0.72x0.64mm_HandSolder" (at 99.06 50.673 90)
+    (property "Footprint" "Resistor_SMD:R_0402_1005Metric" (at 99.06 50.673 90)
       (effects (font (size 1.27 1.27)) hide)
     )
@@
       (effects (font (size 1.27 1.27)) (justify left))
     )
-    (property "Footprint" "Capacitor_SMD:C_0402_1005Metric_Pad0.74x0.62mm_HandSolder" (at 40.9448 180.975 0)
+    (property "Footprint" "Capacitor_SMD:C_0402_1005Metric" (at 40.9448 180.975 0)
       (effects (font (size 1.27 1.27)) hide)
     )
@@
       (effects (font (size 1.27 1.27)) (justify left))
     )
-    (property "Footprint" "Capacitor_SMD:C_0402_1005Metric_Pad0.74x0.62mm_HandSolder" (at 35.8648 149.225 0)
+    (property "Footprint" "Capacitor_SMD:C_0402_1005Metric" (at 35.8648 149.225 0)
       (effects (font (size 1.27 1.27)) hide)
     )
@@
       (effects (font (size 1.27 1.27)) (justify left))
     )
-    (property "Footprint" "Capacitor_SMD:C_0402_1005Metric_Pad0.74x0.62mm_HandSolder" (at 133.6548 180.975 0)
+    (property "Footprint" "Capacitor_SMD:C_0402_1005Metric" (at 133.6548 180.975 0)
       (effects (font (size 1.27 1.27)) hide)
     )
@@
       (effects (font (size 1.27 1.27)))
     )
-    (property "Footprint" "Resistor_SMD:R_0402_1005Metric_Pad0.72x0.64mm_HandSolder" (at 250.19 65.913 90)
+    (property "Footprint" "Resistor_SMD:R_0402_1005Metric" (at 250.19 65.913 90)
       (effects (font (size 1.27 1.27)) hide)
     )
@@
       (effects (font (size 1.27 1.27)) (justify left))
     )
-    (property "Footprint" "Capacitor_SMD:C_0402_1005Metric_Pad0.74x0.62mm_HandSolder" (at 115.8748 180.975 0)
+    (property "Footprint" "Capacitor_SMD:C_0402_1005Metric" (at 115.8748 180.975 0)
       (effects (font (size 1.27 1.27)) hide)
     )
@@
       (effects (font (size 1.27 1.27)))
     )
-    (property "Footprint" "Resistor_SMD:R_0402_1005Metric_Pad0.72x0.64mm_HandSolder" (at 250.19 68.453 90)
+    (property "Footprint" "Resistor_SMD:R_0402_1005Metric" (at 250.19 68.453 90)
       (effects (font (size 1.27 1.27)) hide)
     )
@@
       (effects (font (size 1.27 1.27)) (justify left))
     )
-    (property "Footprint" "Capacitor_SMD:C_0402_1005Metric_Pad0.74x0.62mm_HandSolder" (at 142.5448 180.975 0)
+    (property "Footprint" "Capacitor_SMD:C_0402_1005Metric" (at 142.5448 180.975 0)
       (effects (font (size 1.27 1.27)) hide)
     )
@@
       (effects (font (size 1.27 1.27)) hide)
     )
+    (property "Alternate" "n/a" (at 19.05 98.425 0)
+      (effects (font (size 1.27 1.27)) hide)
+    )
+    (property "Link" "n/a" (at 19.05 98.425 0)
+      (effects (font (size 1.27 1.27)) hide)
+    )
+    (property "Manufacturer" "n/a" (at 19.05 98.425 0)
+      (effects (font (size 1.27 1.27)) hide)
+    )
+    (property "Manufacturer Number" "n/a" (at 19.05 98.425 0)
+      (effects (font (size 1.27 1.27)) hide)
+    )
     (pin "1")
     (pin "2")
@@
       (effects (font (size 1.27 1.27)) hide)
     )
-    (property "Datasheet" "" (at 194.31 107.315 0)
+    (property "Datasheet" "https://datasheets.raspberrypi.com/rp2040/rp2040-datasheet.pdf" (at 194.31 107.315 0)
       (effects (font (size 1.27 1.27)) hide)
     )
@@
       (effects (font (size 1.27 1.27)) (justify left))
     )
-    (property "Footprint" "Capacitor_SMD:C_0402_1005Metric_Pad0.74x0.62mm_HandSolder" (at 160.3248 180.975 0)
+    (property "Footprint" "Capacitor_SMD:C_0402_1005Metric" (at 160.3248 180.975 0)
       (effects (font (size 1.27 1.27)) hide)
     )
@@
       (effects (font (size 1.27 1.27)))
     )
-    (property "Footprint" "Resistor_SMD:R_0402_1005Metric_Pad0.72x0.64mm_HandSolder" (at 99.06 48.133 90)
+    (property "Footprint" "Resistor_SMD:R_0402_1005Metric" (at 99.06 48.133 90)
       (effects (font (size 1.27 1.27)) hide)
     )
@@
       (effects (font (size 1.27 1.27)) (justify left))
     )
-    (property "Footprint" "Capacitor_SMD:C_0402_1005Metric_Pad0.74x0.62mm_HandSolder" (at 44.7548 149.225 0)
+    (property "Footprint" "Capacitor_SMD:C_0402_1005Metric" (at 44.7548 149.225 0)
       (effects (font (size 1.27 1.27)) hide)
     )
@@
       (effects (font (size 1.27 1.27)) (justify left))
     )
-    (property "Footprint" "Capacitor_SMD:C_0402_1005Metric_Pad0.74x0.62mm_HandSolder" (at 169.2148 180.975 0)
+    (property "Footprint" "Capacitor_SMD:C_0402_1005Metric" (at 169.2148 180.975 0)
       (effects (font (size 1.27 1.27)) hide)
     )
@@
       (effects (font (size 1.27 1.27)) (justify left))
     )
-    (property "Footprint" "Capacitor_SMD:C_0402_1005Metric_Pad0.74x0.62mm_HandSolder" (at 124.7648 180.975 0)
+    (property "Footprint" "Capacitor_SMD:C_0402_1005Metric" (at 124.7648 180.975 0)
       (effects (font (size 1.27 1.27)) hide)
     )
@@
       (effects (font (size 1.27 1.27)) (justify left))
     )
-    (property "Footprint" "Capacitor_SMD:C_0402_1005Metric_Pad0.74x0.62mm_HandSolder" (at 151.4348 180.975 0)
+    (property "Footprint" "Capacitor_SMD:C_0402_1005Metric" (at 151.4348 180.975 0)
       (effects (font (size 1.27 1.27)) hide)
     )
@@
       (effects (font (size 1.27 1.27)) (justify left))
     )
-    (property "Footprint" "Capacitor_SMD:C_0402_1005Metric_Pad0.74x0.62mm_HandSolder" (at 16.8148 180.975 0)
+    (property "Footprint" "Capacitor_SMD:C_0402_1005Metric" (at 16.8148 180.975 0)
       (effects (font (size 1.27 1.27)) hide)
     )
@@
       (effects (font (size 1.27 1.27)) (justify left))
     )
-    (property "Footprint" "Capacitor_SMD:C_0402_1005Metric_Pad0.74x0.62mm_HandSolder" (at 106.9848 180.975 0)
+    (property "Footprint" "Capacitor_SMD:C_0402_1005Metric" (at 106.9848 180.975 0)
       (effects (font (size 1.27 1.27)) hide)
     )
@@
       (effects (font (size 1.27 1.27)) (justify left))
     )
-    (property "Footprint" "Capacitor_SMD:C_0402_1005Metric_Pad0.74x0.62mm_HandSolder" (at 26.9748 149.225 0)
+    (property "Footprint" "Capacitor_SMD:C_0402_1005Metric" (at 26.9748 149.225 0)
       (effects (font (size 1.27 1.27)) hide)
     )
@@
       (effects (font (size 1.27 1.27)) (justify left))
     )
-    (property "Footprint" "Capacitor_SMD:C_0402_1005Metric_Pad0.74x0.62mm_HandSolder" (at 49.8348 180.975 0)
+    (property "Footprint" "Capacitor_SMD:C_0402_1005Metric" (at 49.8348 180.975 0)
       (effects (font (size 1.27 1.27)) hide)
     )
@@
       (effects (font (size 1.27 1.27)) (justify left))
     )
-    (property "Footprint" "Capacitor_SMD:C_0402_1005Metric_Pad0.74x0.62mm_HandSolder" (at 16.8148 149.225 0)
+    (property "Footprint" "Capacitor_SMD:C_0402_1005Metric" (at 16.8148 149.225 0)
       (effects (font (size 1.27 1.27)) hide)
     )
@@
       (effects (font (size 1.27 1.27)))
     )
-    (property "Footprint" "Resistor_SMD:R_0402_1005Metric_Pad0.72x0.64mm_HandSolder" (at 139.7 50.673 90)
+    (property "Footprint" "Resistor_SMD:R_0402_1005Metric" (at 139.7 50.673 90)
       (effects (font (size 1.27 1.27)) hide)
     )
@@
       (effects (font (size 1.27 1.27)))
     )
-    (property "Footprint" "Resistor_SMD:R_0402_1005Metric_Pad0.72x0.64mm_HandSolder" (at 139.7 48.133 90)
-      (effects (font (size 1.27 1.27)) hide)
-    )
+    (property "Footprint" "Resistor_SMD:R_0402_1005Metric" (at 139.7 48.133 90)
+      (effects (font (size 1.27 1.27)) hide)
+    )

Commit message: update design notes
Other:
- note added: "Note: Shield is connected to GND1 on PC side."
- note added: "TODO: consider CDDFN2-T5.0LC on VBUS, CC1, CC2"
- note removed: "TODO: CDDFN2-T5.0LC on VBUS, CC1, CC2 TODO: consider connecting shield to GND1 or leaving it disconnected. (This is connected to the PC.)"
Changed lines of the file:
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@@
     (effects (font (size 1.27 1.27)) (justify left bottom))
   )
-  (text "TODO: CDDFN2-T5.0LC on VBUS, CC1, CC2\nTODO: consider connecting shield to GND1 or leaving it disconnected. (This is connected to the PC.)"
-    (at 27.94 -3.175 0)
+  (text "TODO: consider CDDFN2-T5.0LC on VBUS, CC1, CC2\n" (at 27.94 -3.175 0)
     (effects (font (size 2.54 2.54) (thickness 0.508) bold) (justify left bottom))
   )
@@
     (effects (font (size 1.27 1.27)) (justify left bottom))
   )
+  (text "Note: Shield is connected to GND1 on PC side." (at 17.78 76.835 0)
+    (effects (font (size 1.27 1.27)) (justify left bottom))
+  )

Commit message: update footprints; populate bom
Parts:
- R1: footprint Resistor_SMD:R_0402_1005Metric_Pad0.72x0.64mm_HandSolder -> Resistor_SMD:R_0402_1005Metric; Link https://www.digikey.com/en/products/detail/yageo/AC0402FR-1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 -> https://www.digikey.com/en/products/detail/yageo/RT0402BRD0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; Manufacturer Number AC0402FR-131KL -> RT0402BRD071KL; PCBWay Link https://www.pcbway.com/components/detail/AC0402FR131KL/4677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 -> (none)
- R12, R13: footprint Resistor_SMD:R_0603_1608Metric_Pad0.98x0.95mm_HandSolder -> Resistor_SMD:R_0402_1005Metric; Link https://www.digikey.com/en/products/detail/yageo/RC0603FR-0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 -> https://www.digikey.com/en/products/detail/panasonic-electr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; Manufacturer Yageo -> Panasonic Electronic Components; Manufacturer Number RC0603FR-07330RL -> ERA-2AEB331X; Tolerance 1% -> 0.1%
- R8, R9: footprint Resistor_SMD:R_0402_1005Metric_Pad0.72x0.64mm_HandSolder -> Resistor_SMD:R_0402_1005Metric
Other:
- company: (none) -> The Allen Institute for Neural Dynamics
- title: (none) -> Lickety Split Capacitive Lick Detector
Changed lines of the file:
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@@
 (kicad_sch (version 20230121) (generator eeschema)
   (paper "A4")
+  (title_block
+    (title "Lickety Split Capacitive Lick Detector")
+    (date "2023-09-01")
+    (rev "0.5")
+    (company "The Allen Institute for Neural Dynamics")
+  )
   (junction (at 54.61 31.115) (diameter 0) (color 0 0 0 0)
   )
@@
       (effects (font (size 1.27 1.27)) (justify left))
     )
-    (property "Footprint" "Resistor_SMD:R_0402_1005Metric_Pad0.72x0.64mm_HandSolder" (at 245.618 27.305 90)
+    (property "Footprint" "Resistor_SMD:R_0402_1005Metric" (at 245.618 27.305 90)
       (effects (font (size 1.27 1.27)) hide)
     )
@@
       (effects (font (size 1.27 1.27)))
     )
-    (property "Footprint" "Resistor_SMD:R_0603_1608Metric_Pad0.98x0.95mm_HandSolder" (at 260.35 141.478 90)
+    (property "Footprint" "Resistor_SMD:R_0402_1005Metric" (at 260.35 141.478 90)
       (effects (font (size 1.27 1.27)) hide)
     )
-    (property "Datasheet" "https://www.yageo.com/upload/media/product/productsearch/datasheet/rchip/PYu-RC_Group_51_RoHS_L_12.pdf" (at 260.35 139.7 0)
+    (property "Datasheet" "https://industrial.panasonic.com/cdbs/www-data/pdf/RDM0000/AOA0000C307.pdf" (at 260.35 139.7 0)
       (effects (font (size 1.27 1.27)) hide)
     )
-    (property "Link" "https://www.digikey.com/en/products/detail/yageo/RC0603FR-07330RL/727162" (at 260.35 139.7 90)
+    (property "Link" "https://www.digikey.com/en/products/detail/panasonic-electronic-components/ERA-2AEB331X/1705993" (at 260.35 139.7 90)
       (effects (font (size 1.27 1.27)) hide)
     )
-    (property "Manufacturer" "Yageo" (at 260.35 139.7 0)
+    (property "Manufacturer" "Panasonic Electronic Components" (at 260.35 139.7 0)
       (effects (font (size 1.27 1.27)) hide)
     )
-    (property "Manufacturer Number" "RC0603FR-07330RL" (at 260.35 139.7 0)
+    (property "Manufacturer Number" "ERA-2AEB331X" (at 260.35 139.7 0)
       (effects (font (size 1.27 1.27)) hide)
     )
-    (property "Tolerance" "1%" (at 260.35 139.7 0)
+    (property "Tolerance" "0.1%" (at 260.35 139.7 0)
       (effects (font (size 1.27 1.27)) hide)
     )
@@
       (effects (font (size 1.27 1.27)))
     )
-    (property "Footprint" "Resistor_SMD:R_0603_1608Metric_Pad0.98x0.95mm_HandSolder" (at 260.35 135.128 90)
+    (property "Footprint" "Resistor_SMD:R_0402_1005Metric" (at 260.35 135.128 90)
       (effects (font (size 1.27 1.27)) hide)
     )
-    (property "Datasheet" "https://www.yageo.com/upload/media/product/productsearch/datasheet/rchip/PYu-RC_Group_51_RoHS_L_12.pdf" (at 260.35 133.35 0)
+    (property "Datasheet" "https://industrial.panasonic.com/cdbs/www-data/pdf/RDM0000/AOA0000C307.pdf" (at 260.35 133.35 0)
       (effects (font (size 1.27 1.27)) hide)
     )
-    (property "Link" "https://www.digikey.com/en/products/detail/yageo/RC0603FR-07330RL/727162" (at 260.35 133.35 90)
+    (property "Link" "https://www.digikey.com/en/products/detail/panasonic-electronic-components/ERA-2AEB331X/1705993" (at 260.35 133.35 90)
       (effects (font (size 1.27 1.27)) hide)
     )
-    (property "Manufacturer" "Yageo" (at 260.35 133.35 0)
+    (property "Manufacturer" "Panasonic Electronic Components" (at 260.35 133.35 0)
       (effects (font (size 1.27 1.27)) hide)
     )
-    (property "Manufacturer Number" "RC0603FR-07330RL" (at 260.35 133.35 0)
+    (property "Manufacturer Number" "ERA-2AEB331X" (at 260.35 133.35 0)
       (effects (font (size 1.27 1.27)) hide)
     )
-    (property "Tolerance" "1%" (at 260.35 133.35 0)
+    (property "Tolerance" "0.1%" (at 260.35 133.35 0)
       (effects (font (size 1.27 1.27)) hide)
     )
@@
       (effects (font (size 1.27 1.27)))
     )
-    (property "Footprint" "Resistor_SMD:R_0402_1005Metric_Pad0.72x0.64mm_HandSolder" (at 46.99 114.173 90)
+    (property "Footprint" "Resistor_SMD:R_0402_1005Metric" (at 46.99 114.173 90)
       (effects (font (size 1.27 1.27)) hide)
     )
-    (property "Datasheet" "https://www.yageo.com/upload/media/product/productsearch/datasheet/rchip/PYu-AC_51_RoHS_L_10.pdf" (at 46.99 112.395 0)
+    (property "Datasheet" "n/a" (at 46.99 112.395 0)
       (effects (font (size 1.27 1.27)) hide)
     )
@@
       (effects (font (size 1.27 1.27)) hide)
     )
-    (property "Link" "https://www.digikey.com/en/products/detail/yageo/AC0402FR-131KL/14008372" (at 46.99 112.395 90)
+    (property "Link" "https://www.digikey.com/en/products/detail/yageo/RT0402BRD071KL/1069118" (at 46.99 112.395 90)
       (effects (font (size 1.27 1.27)) hide)
     )
@@
       (effects (font (size 1.27 1.27)) hide)
     )
-    (property "Manufacturer Number" "AC0402FR-131KL" (at 46.99 112.395 0)
+    (property "Manufacturer Number" "RT0402BRD071KL" (at 46.99 112.395 0)
       (effects (font (size 1.27 1.27)) hide)
     )
-    (property "PCBWay Link" "https://www.pcbway.com/components/detail/AC0402FR131KL/467737/" (at 46.99 112.395 0)
+    (property "PCBWay Link" "" (at 46.99 112.395 0)
       (effects (font (size 1.27 1.27)) hide)
     )
@@
       (effects (font (size 1.27 1.27)) (justify left))
     )
-    (property "Footprint" "Resistor_SMD:R_0402_1005Metric_Pad0.72x0.64mm_HandSolder" (at 176.53 129.413 90)
+    (property "Footprint" "Resistor_SMD:R_0402_1005Metric" (at 176.53 129.413 90)
       (effects (font (size 1.27 1.27)) hide)
     )

Commit message: consolidate components; add extra decoupling cap to voltage divider
Parts:
- C10, C8, C9: footprint Capacitor_SMD:C_0603_1608Metric -> Capacitor_SMD:C_0402_1005Metric; Link https://www.digikey.com/en/products/detail/samsung-electro-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 -> https://www.digikey.com/en/products/detail/murata-electroni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; Manufacturer Samsung Electro-Mechanics -> Murata Electronics; Manufacturer Number CL10B105KA8NNNC -> GRM155R6YA105KE11J; PCBWay Link https://www.pcbway.com/components/detail/CL10B105KA8NNNC/78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 -> (none); Rated Voltage 25V -> 35V; Temperature Coefficient X7R -> X5R
Changed lines of the file:
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@@
       (effects (font (size 1.27 1.27)) (justify left))
     )
-    (property "Footprint" "Capacitor_SMD:C_0603_1608Metric" (at 60.6552 188.595 0)
-      (effects (font (size 1.27 1.27)) hide)
-    )
-    (property "Datasheet" "https://media.digikey.com/pdf/Data%20Sheets/Samsung%20PDFs/CL10B105KA8NNNC_spec.pdf" (at 59.69 184.785 0)
+    (property "Footprint" "Capacitor_SMD:C_0402_1005Metric" (at 60.6552 188.595 0)
+      (effects (font (size 1.27 1.27)) hide)
+    )
+    (property "Datasheet" "https://search.murata.co.jp/Ceramy/image/img/A01X/G101/ENG/GRM155R6YA105KE11-01.pdf" (at 59.69 184.785 0)
       (effects (font (size 1.27 1.27)) hide)
     )
@@
       (effects (font (size 1.27 1.27)) hide)
     )
-    (property "Link" "https://www.digikey.com/en/products/detail/samsung-electro-mechanics/CL10B105KA8NNNC/3886842" (at 59.69 184.785 0)
-      (effects (font (size 1.27 1.27)) hide)
-    )
-    (property "Manufacturer Number" "CL10B105KA8NNNC" (at 59.69 184.785 0)
-      (effects (font (size 1.27 1.27)) hide)
-    )
-    (property "Manufacturer" "Samsung Electro-Mechanics" (at 59.69 184.785 0)
-      (effects (font (size 1.27 1.27)) hide)
-    )
-    (property "Rated Voltage" "25V" (at 59.69 184.785 0)
-      (effects (font (size 1.27 1.27)) hide)
-    )
-    (property "Temperature Coefficient" "X7R" (at 59.69 184.785 0)
-      (effects (font (size 1.27 1.27)) hide)
-    )
-    (property "PCBWay Link" "https://www.pcbway.com/components/detail/CL10B105KA8NNNC/788079/" (at 59.69 184.785 0)
+    (property "Link" "https://www.digikey.com/en/products/detail/murata-electronics/GRM155R6YA105KE11J/4905163" (at 59.69 184.785 0)
+      (effects (font (size 1.27 1.27)) hide)
+    )
+    (property "Manufacturer Number" "GRM155R6YA105KE11J" (at 59.69 184.785 0)
+      (effects (font (size 1.27 1.27)) hide)
+    )
+    (property "Manufacturer" "Murata Electronics" (at 59.69 184.785 0)
+      (effects (font (size 1.27 1.27)) hide)
+    )
+    (property "Rated Voltage" "35V" (at 59.69 184.785 0)
+      (effects (font (size 1.27 1.27)) hide)
+    )
+    (property "Temperature Coefficient" "X5R" (at 59.69 184.785 0)
+      (effects (font (size 1.27 1.27)) hide)
+    )
+    (property "PCBWay Link" "" (at 59.69 184.785 0)
       (effects (font (size 1.27 1.27)) hide)
     )
@@
       (effects (font (size 1.27 1.27)) (justify left))
     )
-    (property "Footprint" "Capacitor_SMD:C_0603_1608Metric" (at 63.8302 156.845 0)
-      (effects (font (size 1.27 1.27)) hide)
-    )
-    (property "Datasheet" "https://media.digikey.com/pdf/Data%20Sheets/Samsung%20PDFs/CL10B105KA8NNNC_spec.pdf" (at 62.865 153.035 0)
+    (property "Footprint" "Capacitor_SMD:C_0402_1005Metric" (at 63.8302 156.845 0)
+      (effects (font (size 1.27 1.27)) hide)
+    )
+    (property "Datasheet" "https://search.murata.co.jp/Ceramy/image/img/A01X/G101/ENG/GRM155R6YA105KE11-01.pdf" (at 62.865 153.035 0)
       (effects (font (size 1.27 1.27)) hide)
     )
@@
       (effects (font (size 1.27 1.27)) hide)
     )
-    (property "Link" "https://www.digikey.com/en/products/detail/samsung-electro-mechanics/CL10B105KA8NNNC/3886842" (at 62.865 153.035 0)
-      (effects (font (size 1.27 1.27)) hide)
-    )
-    (property "Manufacturer Number" "CL10B105KA8NNNC" (at 62.865 153.035 0)
-      (effects (font (size 1.27 1.27)) hide)
-    )
-    (property "Manufacturer" "Samsung Electro-Mechanics" (at 62.865 153.035 0)
-      (effects (font (size 1.27 1.27)) hide)
-    )
-    (property "Rated Voltage" "25V" (at 62.865 153.035 0)
-      (effects (font (size 1.27 1.27)) hide)
-    )
-    (property "Temperature Coefficient" "X7R" (at 62.865 153.035 0)
-      (effects (font (size 1.27 1.27)) hide)
-    )
-    (property "PCBWay Link" "https://www.pcbway.com/components/detail/CL10B105KA8NNNC/788079/" (at 62.865 153.035 0)
+    (property "Link" "https://www.digikey.com/en/products/detail/murata-electronics/GRM155R6YA105KE11J/4905163" (at 62.865 153.035 0)
+      (effects (font (size 1.27 1.27)) hide)
+    )
+    (property "Manufacturer Number" "GRM155R6YA105KE11J" (at 62.865 153.035 0)
+      (effects (font (size 1.27 1.27)) hide)
+    )
+    (property "Manufacturer" "Murata Electronics" (at 62.865 153.035 0)
+      (effects (font (size 1.27 1.27)) hide)
+    )
+    (property "Rated Voltage" "35V" (at 62.865 153.035 0)
+      (effects (font (size 1.27 1.27)) hide)
+    )
+    (property "Temperature Coefficient" "X5R" (at 62.865 153.035 0)
+      (effects (font (size 1.27 1.27)) hide)
+    )
+    (property "PCBWay Link" "" (at 62.865 153.035 0)
       (effects (font (size 1.27 1.27)) hide)
     )
@@
       (effects (font (size 1.27 1.27)) (justify left))
     )
-    (property "Footprint" "Capacitor_SMD:C_0603_1608Metric" (at 79.7052 188.595 0)
-      (effects (font (size 1.27 1.27)) hide)
-    )
-    (property "Datasheet" "https://media.digikey.com/pdf/Data%20Sheets/Samsung%20PDFs/CL10B105KA8NNNC_spec.pdf" (at 78.74 184.785 0)
+    (property "Footprint" "Capacitor_SMD:C_0402_1005Metric" (at 79.7052 188.595 0)
+      (effects (font (size 1.27 1.27)) hide)
+    )
+    (property "Datasheet" "https://search.murata.co.jp/Ceramy/image/img/A01X/G101/ENG/GRM155R6YA105KE11-01.pdf" (at 78.74 184.785 0)
       (effects (font (size 1.27 1.27)) hide)
     )
@@
       (effects (font (size 1.27 1.27)) hide)
     )
-    (property "Link" "https://www.digikey.com/en/products/detail/samsung-electro-mechanics/CL10B105KA8NNNC/3886842" (at 78.74 184.785 0)
-      (effects (font (size 1.27 1.27)) hide)
-    )
-    (property "Manufacturer Number" "CL10B105KA8NNNC" (at 78.74 184.785 0)
-      (effects (font (size 1.27 1.27)) hide)
-    )
-    (property "Manufacturer" "Samsung Electro-Mechanics" (at 78.74 184.785 0)
-      (effects (font (size 1.27 1.27)) hide)
-    )
-    (property "Rated Voltage" "25V" (at 78.74 184.785 0)
-      (effects (font (size 1.27 1.27)) hide)
-    )
-    (property "Temperature Coefficient" "X7R" (at 78.74 184.785 0)
-      (effects (font (size 1.27 1.27)) hide)
-    )
-    (property "PCBWay Link" "https://www.pcbway.com/components/detail/CL10B105KA8NNNC/788079/" (at 78.74 184.785 0)
-      (effects (font (size 1.27 1.27)) hide)
-    )
+    (property "Link" "https://www.digikey.com/en/products/detail/murata-electronics/GRM155R6YA105KE11J/4905163" (at 78.74 184.785 0)
+      (effects (font (size 1.27 1.27)) hide)
+    )
+    (property "Manufacturer Number" "GRM155R6YA105KE11J" (at 78.74 184.785 0)
+      (effects (font (size 1.27 1.27)) hide)
+    )
+    (property "Manufacturer" "Murata Electronics" (at 78.74 184.785 0)
+      (effects (font (size 1.27 1.27)) hide)
+    )
+    (property "Rated Voltage" "35V" (at 78.74 184.785 0)
+      (effects (font (size 1.27 1.27)) hide)
+    )
+    (property "Temperature Coefficient" "X5R" (at 78.74 184.785 0)
+      (effects (font (size 1.27 1.27)) hide)
+    )
+    (property "PCBWay Link" "" (at 78.74 184.785 0)
+      (effects (font (size 1.27 1.27)) hide)
+    )
