File: hardware/board/harp_lick_detector_capactive/isolated_usb_rp2040.kicad_sch (KiCad schematic)
At the start: 56 parts, among them J2 Conn_01x03_Male, J4 AudioJack3, J5 USB_C_Receptacle_USB2.0, SW2 SW_DIP_x02, U2 TPD2EUSB30, U3 ADUM4160, U4 RP2040, U5 W25Q16JVUXIQ, X1 ECS-TXO-2016

Commit message: add cable drawing
Parts:
- D3: Alternate (none) -> PESD5V0F1BLD,315
Changed lines of the file:
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@@
+			)
+		)
+		(property "Alternate" "PESD5V0F1BLD,315"
+			(at 70.485 23.495 90)
+			(effects
+				(font
+					(size 1.27 1.27)
+				)
+				(hide yes)
 			)
 		)
