File: hardware/board/harp_lick_detector_capactive/lick_detection_afe.kicad_sch (KiCad schematic)
At the start: 37 parts, among them J1 Conn_Coaxial, J3 Conn_Triaxial, U13 ADS7049, U6 LTC6263, U7 LTC6268xS8-10, U8 REF3433QDBVRQ1

Commit message: draft v0.6.0 board
Parts:
- removed C9: 1uF, Capacitor_SMD:C_0402_1005Metric, symbol Device:C
- removed J1: Conn_Coaxial, Connector_Coaxial:SMA_Amphenol_132134-10_Vertical, symbol Connector:Conn_Coaxial
- removed U8: REF3433QDBVRQ1, Package_TO_SOT_SMD:SOT-23-6, symbol Reference_Voltage:REF3233AMDBVREP
- added C30, C31: 150pF, Capacitor_SMD:C_0402_1005Metric, symbol Device:C
- added C59: 100nF, Capacitor_SMD:C_0402_1005Metric, symbol Device:C
- added R26: 102K, Resistor_SMD:R_0402_1005Metric, symbol Device:R
- added R27: 9K53, Resistor_SMD:R_0402_1005Metric, symbol Device:R
- added R46: 124, Resistor_SMD:R_0402_1005Metric, symbol Device:R
- added R47: 127, Resistor_SMD:R_0402_1005Metric, symbol Device:R
- added R48: 9K76, Resistor_SMD:R_0402_1005Metric, symbol Device:R
- added R49, R52: 1K02, Resistor_SMD:R_0402_1005Metric, symbol Device:R
- added TP1: TestPoint, kicad_component_library:TestPoint_Keystone_5027_Miniature, symbol Connector:TestPoint
- added U8: REF2033, Package_TO_SOT_SMD:SOT-23-5, symbol kicad_component_library:REF20xx
- R14: Link https://www.digikey.com/en/products/detail/yageo/RT1206FRE0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 -> RT1206FRE07100KL
- R18: value 49K9 -> 105K; Link https://www.digikey.com/en/products/detail/yageo/RT0402BRE0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 -> https://www.digikey.com/en/products/detail/te-connectivity-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; Manufacturer Yageo -> TE Connectivity Passive Product; Manufacturer Number RT0402BRE0749K9L -> RP73PF1E105KBTD
- R20: value 100K -> 102K; Link https://www.digikey.com/en/products/detail/yageo/RT0402BRD07100KL/1068989 -> https://www.digikey.com/en/products/detail/yageo/RT0402BRD07102KL/1068991; Manufacturer Number RT0402BRD07100KL -> RT0402BRD07102KL
- R21: value 68 -> 102K; Link https://www.digikey.com/en/products/detail/yageo/RT0402BRD0768RL/1069370 -> https://www.digikey.com/en/products/detail/yageo/RT0402BRD07102KL/1068991; Manufacturer Number RT0402BRD0768RL -> RT0402BRD07102KL; Temperature Coefficient 25ppm/C -> (none)
- R22: value 10K -> 102K; Link https://www.digikey.com/en/products/detail/yageo/RT0402BRD0710KL/1068998 -> https://www.digikey.com/en/products/detail/yageo/RT0402BRD07102KL/1068991; Manufacturer Number RT0402BRD0710KL -> RT0402BRD07102KL; Temperature Coefficient 25ppm/C -> (none)
- R23: value 10K -> 105K; Link https://www.digikey.com/en/products/detail/yageo/RT0402BRD0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 -> https://www.digikey.com/en/products/detail/te-connectivity-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; Manufacturer Yageo -> TE Connectivity Passive Product; Manufacturer Number RT0402BRD0710KL -> RP73PF1E105KBTD; Temperature Coefficient 25ppm/C -> (none)
- R24: value 10K -> 1K05; Link https://www.digikey.com/en/products/detail/yageo/RT0402BRD0710KL/1068998 -> https://www.digikey.com/en/products/detail/yageo/RT0402BRD071K05L/1069088; Manufacturer Number RT0402BRD0710KL -> RT0402BRD071K05L; Temperature Coefficient 25ppm/C -> (none)
- R42, R43: value 16 -> 68; Link https://www.digikey.com/en/products/detail/yageo/RC0402FR-0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 -> https://www.digikey.com/en/products/detail/yageo/RT0402BRD0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; Manufacturer Number RC0402FR-0716RL -> RT0402BRD0768RL; Temperature Coefficient (none) -> 25ppm/C; Tolerance 1% -> 0.1%
- renumbered C30 to C33, C31 to C34
Connections:
- net +5V: now also U8.3 (EN), U8.4 (VIN)
- net GND: now also R24.1, R42.1, C59.1, R46.1, R47.1, R52.2, U8.2 (GND); no longer R42.2, U6.14 (+), U6.5 (+)
- net VREF_3V3: now also U8.5 (VREF); no longer C38.2, R23.2
- net at C52.2, U13.5 (AINM): now also R42.2; no longer R42.1
- net at C52.1, U13.6 (AINP): now also R43.1; no longer R43.2
- net at C33.1, C34.1: now also R23.2, R24.2; no longer R18.2, R19.2
- net at R20.2, U6.7: now also R23.1, C30.2, R27.2; no longer C33.2, R21.1
- net at R20.1, U6.6 (-): now also C31.2; no longer C34.2
- new net: R21.1, R49.1, U6.12 (+)
- new net: C33.2, R26.2, R48.2, R49.2, U6.16
- new net: R22.2, R52.1, U6.11 (-)
- new net: R22.1, R43.2, TP1.1, U6.10
- new net: R47.2, R48.1, U6.14 (+)
- new net: C34.2, R26.1, U6.15 (-)
- new net: C30.1, C31.1, R18.2, R19.2
- new net: R27.1, R46.2, U6.5 (+)
- new net VREF_1V65: C38.2, C59.2, R21.2, U8.1 (VBIAS)
Other:
- note added: "100x Inverting Amplification +1.65V DC offset"
- note added: "4th Order Bandpass Filter"
- note added: "Mouse body: < 100pF"
- note added: "Note: test point output will look slightly distorted with small transient spikes when the ADS7049 is acquiring samples."
- note added: "Note: this setup must be grounded to the animal at a single point using either H1 or the outer shield of J3's cable. (i.e: current must flow out of the lick detector water delivery spout, through the animal's tongue, to ground. The sensing element is connected to a conductive water delivery spout.)"
- note added: "Place C38 near R21."
- note added: "R14 = 100K, Ctotal = 0.1pF, Vout = 99%Vin R14 = 100K, Ctotal = 1pF, Vout = 94%Vin R14 = 100K, Ctotal = 5pF, Vout = 76%Vin R14 = 100K, Ctotal = 10pF, Vout = 61%Vin R14 = 100K, Ctotal = 50pF, Vout = 24%Vin"
- note added: "REF2033 Bypass Caps"
- note added: "Sensing Analog Front End"
- note removed: "147x Inverting Amplification"
- note removed: "Inverting 2nd Order Bandpass Filter"
- note removed: "Mouse body: ~100pF"
- note removed: "Note: this setup must be grounded to the rig at a single point using H1."
- note removed: "Place C38 near R23."
- note removed: "R23 = 100K, Ctotal = 0.1pF, Vout = 99%Vin R23 = 100K, Ctotal = 1pF, Vout = 94%Vin R23 = 100K, Ctotal = 5pF, Vout = 76%Vin R23 = 100K, Ctotal = 10pF, Vout = 61%Vin R23 = 100K, Ctotal = 50pF, Vout = 24%Vin"
- note removed: "REF3433 Bypass Caps"
- note removed: "Sensing Front End"
- note removed: "Vout = Vsignal/2 + 1.65VDC"
- moved on the sheet: C24, C25, C26, C28, C33, C34, C38, C8, C9, J3, R14, R15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

Commit message: make r0.6 board snapshot
Parts:
- C22, C23: Alternate (none) -> CL21B106KOQNNNE
Other:
- note added: "TODO: consider REF2025 so we don't get clipping from the +/-2.5V supply of the LTC6263."
Changed lines of the file:
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@@
     (effects (font (size 2 2) (thickness 0.254) bold) (justify left bottom))
+  )
+  (text "TODO: consider REF2025\nso we don't get clipping\nfrom the +/-2.5V supply of the\nLTC6263."
+    (at 201.295 36.83 0)
+    (effects (font (size 1.27 1.27) (thickness 0.254) bold) (justify left bottom))
   )
   (text "Note: LTC6268 and LTC6263 inputs are ESD protected."
@@
     )
     (property "Tolerance" "" (at 32.385 172.72 0)
+      (effects (font (size 1.27 1.27)) hide)
+    )
+    (property "Alternate" "CL21B106KOQNNNE" (at 32.385 172.72 0)
       (effects (font (size 1.27 1.27)) hide)
     )
@@
       (effects (font (size 1.27 1.27)) hide)
     )
+    (property "Alternate" "CL21B106KOQNNNE" (at 32.385 184.15 0)
+      (effects (font (size 1.27 1.27)) hide)
+    )
