File: hardware/board/harp_lick_detector_capactive/harp_lick_detector_capactive.kicad_sch (KiCad schematic)
At the start: 0 parts

Commit message: draft v0.7 pcb schematic and layout
Other:
- sheet 100KHz Sine Wave ports: added 100KHZ_IN, 125KHZ_IN; removed 100KHZ_SQ_WAVE_IN
- sheet Harp Core RP2040 + Isolated USB ports: added 100KHZ_OUT, 125KHZ_OUT; removed 100KHZ_SQ_WAVE_OUT
- note added: "Device Functionality Options: * 100 or 125KHz excitation signal frequency. * for multiple lick detectors with lick tubes spaced <10mm apart. * 20mVpp or 2Vpp excitation signal amplitude * (1) for Ephys and (2) general purpose setups."
Changed lines of the file:
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@@
+    (stroke (width 0) (type default))
+  )
+  (wire (pts (xy 118.745 83.185) (xy 169.545 83.185))
     (stroke (width 0) (type default))
   )
@@
   (wire (pts (xy 118.745 85.725) (xy 169.545 85.725))
     (stroke (width 0) (type default))
+  )
+  (text "Device Functionality Options:\n\n* 100 or 125KHz excitation signal frequency.\n  * for multiple lick detectors with lick tubes spaced <10mm apart.\n* 20mVpp or 2Vpp excitation signal amplitude\n  * (1) for Ephys and (2) general purpose setups."
+    (at 16.51 191.77 0)
+    (effects (font (size 2 2) (thickness 0.254) bold) (justify left bottom))
   )
   (sheet (at 207.645 86.36) (size 13.97 14.605) (fields_autoplaced)
@@
     )
   )
-  (sheet (at 94.615 81.28) (size 24.13 26.035) (fields_autoplaced)
+  (sheet (at 94.615 80.01) (size 24.13 27.305) (fields_autoplaced)
     (stroke (width 0.1524) (type solid))
     (fill (color 0 0 0 0.0000))
-    (property "Sheetname" "100KHz Sine Wave" (at 94.615 80.5684 0)
+    (property "Sheetname" "100KHz Sine Wave" (at 94.615 79.2984 0)
       (effects (font (size 1.27 1.27)) (justify left bottom))
     )
@@
       (effects (font (size 1.27 1.27)) (justify right))
     )
-    (pin "100KHZ_SQ_WAVE_IN" input (at 118.745 85.725 0)
+    (pin "125KHZ_IN" input (at 118.745 83.185 0)
+      (effects (font (size 1.27 1.27)) (justify right))
+    )
+    (pin "100KHZ_IN" input (at 118.745 85.725 0)
       (effects (font (size 1.27 1.27)) (justify right))
     )
@@
     )
   )
-  (sheet (at 133.35 95.25) (size 20.32 12.065) (fields_autoplaced)
+  (sheet (at 133.35 90.805) (size 20.32 16.51) (fields_autoplaced)
     (stroke (width 0.1524) (type solid))
     (fill (color 0 0 0 0.0000))
-    (property "Sheetname" "Lick Detection Analog Front End" (at 133.35 94.5384 0)
+    (property "Sheetname" "Lick Detection Analog Front End" (at 133.35 90.0934 0)
       (effects (font (size 1.27 1.27)) (justify left bottom))
     )
@@
       (effects (font (size 1.27 1.27)) (justify left))
     )
-    (pin "100KHZ_SQ_WAVE_OUT" input (at 169.545 85.725 180)
+    (pin "100KHZ_OUT" input (at 169.545 85.725 180)
       (effects (font (size 1.27 1.27)) (justify left))
     )
+    (pin "125KHZ_OUT" input (at 169.545 83.185 180)
+      (effects (font (size 1.27 1.27)) (justify left))
+    )
