File: hardware/board/harp_lick_detector_capactive/function_generator.kicad_sch (KiCad schematic)
At the start: 19 parts, among them U16 AD8615, U18 TS5A9411DCKR

Commit message: implement soe feedback in layout
Parts:
- R50: Link https://www.digikey.com/en/products/detail/koa-speer-electr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 -> https://www.digikey.com/en/products/detail/yageo/RT0402BRE0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; Manufacturer KOA Speer Electronics, Inc. -> Yageo; Manufacturer Number RN73R1ETTP2201B25 -> RT0402BRE072K2L; Vendor Number 2019-RN73R1ETTP2201B25CT-ND -> (none)
- U16: Link (none) -> https://www.digikey.com/en/products/detail/analog-devices-i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; Manufacturer (none) -> Analog Devices Inc.; Manufacturer Number (none) -> AD8615AUJZ-R2
- U18: Link (none) -> https://www.digikey.com/en/products/detail/texas-instrument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; Manufacturer (none) -> Texas Instruments; Manufacturer Number (none) -> TS5A9411DCKR
Changed lines of the file:
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@@
+      (effects (font (size 1.27 1.27)) hide)
+    )
+    (property "Link" "https://www.digikey.com/en/products/detail/texas-instruments/TS5A9411DCKR/1739550" (at 162.56 120.015 0)
+      (effects (font (size 1.27 1.27)) hide)
+    )
+    (property "Manufacturer" "Texas Instruments" (at 162.56 120.015 0)
+      (effects (font (size 1.27 1.27)) hide)
+    )
+    (property "Manufacturer Number" "TS5A9411DCKR" (at 162.56 120.015 0)
       (effects (font (size 1.27 1.27)) hide)
     )
@@
       (effects (font (size 1.27 1.27)) hide)
     )
-    (property "Datasheet" "https://www.koaspeer.com/pdfs/RN73R.pdf" (at 86.36 99.06 0)
-      (effects (font (size 1.27 1.27)) hide)
-    )
-    (property "Link" "https://www.digikey.com/en/products/detail/koa-speer-electronics-inc/RN73R1ETTP2201B25/10002346" (at 86.36 99.06 0)
-      (effects (font (size 1.27 1.27)) hide)
-    )
-    (property "Manufacturer" "KOA Speer Electronics, Inc." (at 86.36 99.06 0)
-      (effects (font (size 1.27 1.27)) hide)
-    )
-    (property "Manufacturer Number" "RN73R1ETTP2201B25" (at 86.36 99.06 0)
+    (property "Datasheet" "https://www.yageo.com/upload/media/product/app/datasheet/rchip/pyu-rt_1-to-0.01_rohs_l.pdf" (at 86.36 99.06 0)
+      (effects (font (size 1.27 1.27)) hide)
+    )
+    (property "Link" "https://www.digikey.com/en/products/detail/yageo/RT0402BRE072K2L/1069637" (at 86.36 99.06 0)
+      (effects (font (size 1.27 1.27)) hide)
+    )
+    (property "Manufacturer" "Yageo" (at 86.36 99.06 0)
+      (effects (font (size 1.27 1.27)) hide)
+    )
+    (property "Manufacturer Number" "RT0402BRE072K2L" (at 86.36 99.06 0)
       (effects (font (size 1.27 1.27)) hide)
     )
     (property "Tolerance" "0.1%" (at 86.36 99.06 0)
-      (effects (font (size 1.27 1.27)) hide)
-    )
-    (property "Vendor Number" "2019-RN73R1ETTP2201B25CT-ND" (at 86.36 99.06 0)
       (effects (font (size 1.27 1.27)) hide)
     )
@@
       (effects (font (size 1.27 1.27)) hide)
     )
+    (property "Link" "https://www.digikey.com/en/products/detail/analog-devices-inc/AD8615AUJZ-R2/993310" (at 162.56 99.06 0)
+      (effects (font (size 1.27 1.27)) hide)
+    )
+    (property "Manufacturer" "Analog Devices Inc." (at 162.56 99.06 0)
+      (effects (font (size 1.27 1.27)) hide)
+    )
+    (property "Manufacturer Number" "AD8615AUJZ-R2" (at 162.56 99.06 0)
+      (effects (font (size 1.27 1.27)) hide)
+    )
     (pin "2")
     (pin "5")
@@
       (effects (font (size 1.27 1.27)) hide)
     )
+    (property "Link" "https://www.digikey.com/en/products/detail/texas-instruments/TS5A9411DCKR/1739550" (at 100.33 178.435 0)
+      (effects (font (size 1.27 1.27)) hide)
+    )
+    (property "Manufacturer" "Texas Instruments" (at 100.33 178.435 0)
+      (effects (font (size 1.27 1.27)) hide)
+    )
+    (property "Manufacturer Number" "TS5A9411DCKR" (at 100.33 178.435 0)
+      (effects (font (size 1.27 1.27)) hide)
+    )

Commit message: draft v0.8 pcb layout
Parts:
- removed U18: TS5A9411DCKR, Package_TO_SOT_SMD:SOT-363_SC-70-6, symbol kicad_component_library:TS5A9411DCKR
- added C20: 100nF, Capacitor_SMD:C_0402_1005Metric, symbol Device:C
- added U18: MAX4564EKA, Package_TO_SOT_SMD:SOT-23-8, symbol kicad_component_library:MAX4564EKA+T
Connections:
- net +3V3 is gone; now on net +2V5: C20.2
- net +2V5: now also U18.2 (V+)
- net -2V5: now also C20.2, U18.6 (V-)
- net GND: now also C20.1, U18.5 (GND), U18.7 (~{EN})
- net at R49.1: now also U18.1
- net at U16.4 (-): now also U18.8
- net at R21.1, R49.1: now also U18.4
- new net GAIN_SEL_2V5: U18.3
Other:
- note added: "U18 Bypass Caps"
- note removed: "U18 Bypass Cap"
- moved on the sheet: C20

Commit message: v0.8 pcb draft ready; schematic components up to date
Parts:
- removed U16: AD8615, Package_TO_SOT_SMD:TSOT-23-5, symbol kicad_component_library:AD8615
- added U17: ADA4891-1, Package_TO_SOT_SMD:SOT-23-5, symbol kicad_component_library:ADA4891-1
Connections:
- net +2V5: now also U17.5 (V+)
- net -2V5: now also U17.2 (V-)
- net VSINE: now also U17.1
- net at C10.2, R25.1: now also U17.3 (+)
- net at U18.8: now also U17.4 (-)
Changed lines of the file:
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@@
+    )
+  )
+  (symbol (lib_id "kicad_component_library:ADA4891-1") (at 162.56 99.06 0) (unit 1)
+    (in_bom yes) (on_board yes) (dnp no)
+    (property "Reference" "U17" (at 163.83 102.87 0)
+      (effects (font (size 1.27 1.27)))
+    )
+    (property "Value" "ADA4891-1" (at 166.37 94.615 0)
+      (effects (font (size 1.27 1.27)))
+    )
+    (property "Footprint" "Package_TO_SOT_SMD:SOT-23-5" (at 162.56 99.06 0)
+      (effects (font (size 1.27 1.27)) hide)
+    )
+    (property "Datasheet" "https://www.analog.com/media/en/technical-documentation/data-sheets/ADA4891-1_4891-2_4891-3_4891-4.PDF" (at 162.56 93.98 0)
+      (effects (font (size 1.27 1.27)) hide)
+    )
+    (property "Manufacturer" "Analog Devices Inc." (at 162.56 99.06 0)
+      (effects (font (size 1.27 1.27)) hide)
+    )
+    (property "Manufacturer Number" "ADA4891-1ARJZ-R7" (at 162.56 99.06 0)
+      (effects (font (size 1.27 1.27)) hide)
+    )
+    (property "Link" "https://www.digikey.com/en/products/detail/analog-devices-inc/ADA4891-1ARJZ-R7/2342630" (at 162.56 99.06 0)
+      (effects (font (size 1.27 1.27)) hide)
+    )
+    (pin "2")
+    (pin "5")
+    (pin "1")
+    (pin "3")
+    (pin "4")
+    (instances
+      (project "harp_lick_detector_capactive"
+        (path "/e63e39d7-6ac0-4ffd-8aa3-1841a4541b55/4df88917-387d-4e6a-a0c2-9efea845a08d"
+          (reference "U17") (unit 1)
+        )
+      )
     )
   )
@@
         )
       )
-    )
-  )
-  (symbol (lib_id "kicad_component_library:AD8615") (at 162.56 99.06 0) (unit 1)
-    (in_bom yes) (on_board yes) (dnp no)
-    (property "Reference" "U16" (at 166.37 93.98 0)
-      (effects (font (size 1.27 1.27)))
-    )
-    (property "Value" "AD8615" (at 168.275 95.885 0)
-      (effects (font (size 1.27 1.27)))
-    )
-    (property "Footprint" "Package_TO_SOT_SMD:TSOT-23-5" (at 162.56 99.06 0)
-      (effects (font (size 1.27 1.27)) hide)
-    )
-    (property "Datasheet" "https://www.analog.com/media/en/technical-documentation/data-sheets/AD8615_8616_8618.pdf" (at 162.56 93.98 0)
-      (effects (font (size 1.27 1.27)) hide)
-    )
-    (property "Link" "https://www.digikey.com/en/products/detail/analog-devices-inc/AD8615AUJZ-R2/993310" (at 162.56 99.06 0)
-      (effects (font (size 1.27 1.27)) hide)
-    )
-    (property "Manufacturer" "Analog Devices Inc." (at 162.56 99.06 0)
-      (effects (font (size 1.27 1.27)) hide)
-    )
-    (property "Manufacturer Number" "AD8615AUJZ-R2" (at 162.56 99.06 0)
-      (effects (font (size 1.27 1.27)) hide)
-    )
-    (pin "2")
-    (pin "5")
-    (pin "1")
-    (pin "3")
-    (pin "4")
-    (instances
-      (project "harp_lick_detector_capactive"
-        (path "/e63e39d7-6ac0-4ffd-8aa3-1841a4541b55/8b2c79bc-d662-4528-ac6e-e4616ba8e8ad"
-          (reference "U16") (unit 1)
-        )
-        (path "/e63e39d7-6ac0-4ffd-8aa3-1841a4541b55/4df88917-387d-4e6a-a0c2-9efea845a08d"
-          (reference "U17") (unit 1)
-        )
-      )
