File: hardware/board/harp_lick_detector_capactive/function_generator.kicad_sch (KiCad schematic)
At the start: 20 parts, among them U17 ADA4891-1, U18 MAX4564EKA

Commit message: finish rev8
Parts:
- U18: Link (none) -> https://www.digikey.com/en/products/detail/analog-devices-i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; Manufacturer (none) -> Analog Devices Inc./Maxim Integrated; Manufacturer Number (none) -> MAX4564EKA+T
Changed lines of the file:
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@@
+      (effects (font (size 1.27 1.27)) hide)
+    )
+    (property "Link" "https://www.digikey.com/en/products/detail/analog-devices-inc-maxim-integrated/MAX4564EKA-T/1781971" (at 162.56 122.555 0)
+      (effects (font (size 1.27 1.27)) hide)
+    )
+    (property "Manufacturer" "Analog Devices Inc./Maxim Integrated" (at 162.56 122.555 0)
+      (effects (font (size 1.27 1.27)) hide)
+    )
+    (property "Manufacturer Number" "MAX4564EKA+T" (at 162.56 122.555 0)
       (effects (font (size 1.27 1.27)) hide)
     )
@@
       (effects (font (size 1.27 1.27)) hide)
     )
+    (property "Link" "https://www.digikey.com/en/products/detail/analog-devices-inc-maxim-integrated/MAX4564EKA-T/1781971" (at 125.73 179.07 0)
+      (effects (font (size 1.27 1.27)) hide)
+    )
+    (property "Manufacturer" "Analog Devices Inc./Maxim Integrated" (at 125.73 179.07 0)
+      (effects (font (size 1.27 1.27)) hide)
+    )
+    (property "Manufacturer Number" "MAX4564EKA+T" (at 125.73 179.07 0)
+      (effects (font (size 1.27 1.27)) hide)
+    )

Commit message: update to new harp core
Parts:
- renumbered C10 to C32, C10 to C35, C10 to C36, C10 to C57, C10 to C58, C20 to C61, C21 to C62, C20 to C63, C20 to C71, R49 to R54, R21 to R55, R49 to R56
