File: hardware/board/harp_lick_detector_capactive/board_power.kicad_sch (KiCad schematic)
At the start: 25 parts, among them J5 Barrel_Jack_Switch, U5 LT3030, U6 LM27762

Commit message: v0.8 pcb draft ready; schematic components up to date
Parts:
- U5: symbol machine_agency_components:LT3030 -> kicad_component_library:LT3030
Changed lines of the file:
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@@
     )
   )
-  (symbol (lib_id "machine_agency_components:LT3030") (at 133.35 59.69 0) (unit 1)
+  (symbol (lib_id "kicad_component_library:LT3030") (at 133.35 59.69 0) (unit 1)
     (in_bom yes) (on_board yes) (dnp no)
     (property "Reference" "U5" (at 125.73 45.72 0)

Commit message: update to new harp core
Parts:
- added C76, C77: 10uF, Capacitor_SMD:C_0805_2012Metric, symbol Device:C
- renumbered C5 to C40, C6 to C41, C7 to C42, C8 to C43, C8 to C44, C1 to C45, C32 to C46, C32 to C47, C4 to C48, C5 to C49, C1 to C67, J5 to J6, R11 to R32, R13 to R33, R12 to R34, R14 to R35, R2 to R36, R2 to R37, R52 to R38, R62 to R39, R20 to R40, R20 to R41, U6 to U11, U5 to U12
Connections:
- net +2V5: now also C76.2
- net -2V5: now also C77.2
- net GND: now also C76.1, C77.1
Other:
- moved on the sheet: C45, C46, C47, C48, C49, C67, J6, L1, R36, R37, R38, R39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
