File: hardware/board/square_wave_filter_scheme/square_wave_filter_scheme/square_wave_filter_scheme.kicad_sch (KiCad schematic)
At the start: 11 parts

Commit message: draft v0.7 pcb schematic and layout
Other:
- note added: "Use 2.2K for R1 in 125KHz configuration."
Changed lines of the file:
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@@
     (stroke (width 0) (type default))
+  )
+  (text "Use 2.2K for R1 in 125KHz configuration." (at 88.265 149.225 0)
+    (effects (font (size 1.27 1.27)) (justify left bottom))
   )
   (global_label "OUT" (shape input) (at 178.435 112.395 0) (fields_autoplaced)
@@
       (effects (font (size 1.27 1.27)) (justify left) hide)
     )
-    (property "Sim.Params" "y1=0 y2=3.3 td=2n tr=2n tf=2n tw=5u per=10u" (at 54.61 134.62 0)
+    (property "Sim.Params" "y1=0 y2=3.3 td=2n tr=2n tf=2n tw=4u per=8u" (at 54.61 134.62 0)
       (effects (font (size 1.27 1.27)) (justify left))
     )
