File: hardware/board/main_board/sma_ttl_out.kicad_sch (KiCad schematic)
At the start: 8 parts, among them J7 Conn_Coaxial, U1 74LVCH2T45DC

Commit message: split board into two
Connections:
- net +3.3V renamed +3V3
Other:
- moved on the sheet: C53, J7, R30, R31, U1

Commit message: update buffer board soldermask cutout
Parts:
- C39: Alternate CL21B106KOQNNNE -> (none)
Changed lines of the file:
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@@
 			)
 		)
-		(property "Alternate" "CL21B106KOQNNNE"
+		(property "Alternate" ""
 			(at 154.94 179.07 0)
 			(effects
